File: Hardware/keyboard.sch (KiCad schematic (older format))
At the start: 139 parts

Commit message: Remove Tracks
Parts:
- added C1: 1uF, Capacitor_SMD:C_0805_2012Metric, symbol Device:C_Small
- added C2, C3, C4: 0.1uF, Capacitor_SMD:C_0805_2012Metric, symbol Device:C_Small
- added C5: 10uF, Capacitor_SMD:C_0805_2012Metric, symbol Device:C_Small
- added F1: 500mA, Fuse:Fuse_1206_3216Metric, symbol Device:Polyfuse_Small
- added J1: USB2_C_Receptacle, usb-type-c:Mid_Mount-USB_C_HandSoldering, symbol usb-type-c:USB2_C_Receptacle
- added R1, R6: 10k, Resistor_SMD:R_0805_2012Metric, symbol Device:R_Small
- added R2, R3: 5.1k, Resistor_SMD:R_0805_2012Metric, symbol Device:R_Small
- added R4, R5: 22, Resistor_SMD:R_0805_2012Metric, symbol Device:R_Small
- added SW1: SW_Push, random-keyboard-parts:SKQG-1155865, symbol Switch:SW_Push
- added U1: ATmega32U4-AU, Package_QFP:TQFP-44_10x10mm_P0.8mm, symbol MCU_Microchip_ATmega:ATmega32U4-AU
- added U2: SRV05-4, Package_TO_SOT_SMD:SOT-23-6, symbol Power_Protection:SRV05-4
- added Y1: 16MHz, proj_local:Resonator_SMD_muRata_CSTxExxV-3Pin_3.0x1.1mm_HandSoldering_Compact, symbol Device:Resonator_Small
Connections:
- new net: R1.2, SW1.2, U1.13 (~RESET)
- new net: U1.16 (XTAL2), Y1.3
- new net: U1.17 (XTAL1), Y1.1
- new net: R5.1, U1.3 (D-)
- new net: R6.2, U1.33 (~HWB~/PE2)
- new net: R4.1, U1.4 (D+)
- new net: C1.1, U1.6 (UCAP)
- new net: J1.A5 (CC1), R2.2
- new net: J1.B5 (CC2), R3.2
- new net +5V: C2.1, C3.1, C4.1, C5.1, F1.1, R1.1, U1.14 (VCC), U1.2 (UVCC), U1.24 (AVCC), U1.34 (VCC), U1.44 (AVCC), U1.7 (VBUS)
- new net D+: J1.A6 (D+), J1.B6 (D+), R4.2, U2.6 (IO4)
- new net D-: J1.A7 (D-), J1.B7 (D-), R5.2, U2.1 (IO1)
- new net GND: C1.2, C2.2, C3.2, C4.2, C5.2, J1.A1B12 (GND), J1.B1A12 (GND), J1.S1 (Shield), R2.1, R3.1, R6.1, SW1.1, U1.15 (GND), U1.23 (GND), U1.35 (GND), U1.43 (GND), U1.5 (UGND), U2.2 (VN), Y1.2
- new net VCC: F1.2, J1.A4B9 (VBUS), J1.B4A9 (VBUS), U2.5 (VP)

Commit message: Add Encoders
Parts:
- added SW2, SW3, SW4: Rotary_Encoder_Switch, Keebio-Parts:RotaryEncoder_EC11, symbol Device:Rotary_Encoder_Switch
Connections:
- net GND: now also SW2.C, SW3.C, SW4.C
- net 1row: now reaches D_30.2 (A), K_30.2 (ROW)
- net 1row: now also SW3.S1
- net 2row: now reaches D_44.2 (A), K_45.2 (ROW)
- net 2row: now also SW4.S1
- net 0row: now reaches D_15.2 (A), K_15.2 (ROW)
- net 0row: now also SW2.S1
- net col14 renamed 0col
- net 0col: now also SW2.S2, SW3.S2, SW4.S2
- new net ENC0A: SW2.A
- new net ENC1A: SW3.A
- new net ENC2A: SW4.A
- new net ENCB: SW2.B, SW3.B, SW4.B
Changed lines of the file:
@@
 Connection ~ 17900 9800
-$Comp
-L MX_Alps_Hybrid:MX-NoLED K_15
-U 1 1 00000051
-P 18950 9400
-F 0 "K_15" H 18950 9633 60  0000 C CNN
-F 1 "KEYSW" H 18950 9300 60  0001 C CNN
-F 2 "MX_Only:MXOnly-1U-NoLED" H 18950 9400 60  0001 C CNN
-F 3 "" H 18950 9400 60  0000 C CNN
-	1    18950 9400
-	1    0    0    -1
-$EndComp
 $Comp
 L Device:D_Small D_15
@@
 Connection ~ 17900 10800
 $Comp
-L MX_Alps_Hybrid:MX-NoLED K_30
-U 1 1 00000121
-P 18950 10400
-F 0 "K_30" H 18950 10633 60  0000 C CNN
-F 1 "KEYSW" H 18950 10300 60  0001 C CNN
-F 2 "MX_Only:MXOnly-1U-NoLED" H 18950 10400 60  0001 C CNN
-F 3 "" H 18950 10400 60  0000 C CNN
-	1    18950 10400
-	1    0    0    -1
-$EndComp
-$Comp
 L Device:D_Small D_30
 U 1 1 00000120
@@
 Connection ~ 17900 11800
 $Comp
-L MX_Alps_Hybrid:MX-NoLED K_45
-U 1 1 00000181
-P 18950 11400
-F 0 "K_45" H 18950 11633 60  0000 C CNN
-F 1 "KEYSW" H 18950 11300 60  0001 C CNN
-F 2 "MX_Only:MXOnly-1U-NoLED" H 18950 11400 60  0001 C CNN
-F 3 "" H 18950 11400 60  0000 C CNN
-	1    18950 11400
-	1    0    0    -1
-$EndComp
-$Comp
 L Device:D_Small D_44
 U 1 1 00000180
@@
 $EndComp
 $Comp
-L power:GND #PWR017
+L power:GND #PWR016
 U 1 1 5EA13457
 P 4700 6000
-F 0 "#PWR017" H 4700 5750 50  0001 C CNN
+F 0 "#PWR016" H 4700 5750 50  0001 C CNN
 F 1 "GND" H 4705 5827 50  0000 C CNN
 F 2 "" H 4700 6000 50  0001 C CNN
@@
 	3900 4100 3900 4300
 $Comp
-L power:GND #PWR012
+L power:GND #PWR011
 U 1 1 5EA2C83C
 P 3900 4300
-F 0 "#PWR012" H 3900 4050 50  0001 C CNN
+F 0 "#PWR011" H 3900 4050 50  0001 C CNN
 F 1 "GND" H 3905 4127 50  0000 C CNN
 F 2 "" H 3900 4300 50  0001 C CNN
@@
 	3650 2600 3100 2600
 $Comp
-L power:GND #PWR06
+L power:GND #PWR03
 U 1 1 5EAC4999
 P 3100 2600
-F 0 "#PWR06" H 3100 2350 50  0001 C CNN
+F 0 "#PWR03" H 3100 2350 50  0001 C CNN
 F 1 "GND" H 3105 2427 50  0000 C CNN
 F 2 "" H 3100 2600 50  0001 C CNN
@@
 	6650 4700 7000 4700
 $Comp
-L power:GND #PWR013
+L power:GND #PWR012
 U 1 1 5EC6CA51
 P 7000 4700
-F 0 "#PWR013" H 7000 4450 50  0001 C CNN
+F 0 "#PWR012" H 7000 4450 50  0001 C CNN
 F 1 "GND" H 7005 4527 50  0000 C CNN
 F 2 "" H 7000 4700 50  0001 C CNN
@@
 	3200 5300 3400 5300
 $Comp
-L power:+5V #PWR014
+L power:+5V #PWR013
 U 1 1 5ED653F9
 P 3200 5000
-F 0 "#PWR014" H 3200 4850 50  0001 C CNN
+F 0 "#PWR013" H 3200 4850 50  0001 C CNN
 F 1 "+5V" H 3215 5173 50  0000 C CNN
 F 2 "" H 3200 5000 50  0001 C CNN
@@
 $EndComp
 $Comp
-L power:GND #PWR015
+L power:GND #PWR014
 U 1 1 5ED66198
 P 3200 5400
-F 0 "#PWR015" H 3200 5150 50  0001 C CNN
+F 0 "#PWR014" H 3200 5150 50  0001 C CNN
 F 1 "GND" H 3205 5227 50  0000 C CNN
 F 2 "" H 3200 5400 50  0001 C CNN
@@
 $EndComp
 $Comp
-L power:GND #PWR010
+L power:GND #PWR07
 U 1 1 5EEC6D34
 P 8450 2950
-F 0 "#PWR010" H 8450 2700 50  0001 C CNN
+F 0 "#PWR07" H 8450 2700 50  0001 C CNN
 F 1 "GND" H 8455 2777 50  0000 C CNN
 F 2 "" H 8450 2950 50  0001 C CNN
@@
 $EndComp
 $Comp
-L power:GND #PWR07
+L power:GND #PWR06
 U 1 1 5EEC7B66
 P 8550 2850
-F 0 "#PWR07" H 8550 2600 50  0001 C CNN
+F 0 "#PWR06" H 8550 2600 50  0001 C CNN
 F 1 "GND" H 8555 2677 50  0000 C CNN
 F 2 "" H 8550 2850 50  0001 C CNN
@@
 D+ESD
 $Comp
-L power:GND #PWR016
+L power:GND #PWR015
 U 1 1 5F039596
 P 8600 5650
-F 0 "#PWR016" H 8600 5400 50  0001 C CNN
+F 0 "#PWR015" H 8600 5400 50  0001 C CNN
 F 1 "GND" H 8605 5477 50  0000 C CNN
 F 2 "" H 8600 5650 50  0001 C CNN
@@
 	7150 4000 7150 4150
 $Comp
-L power:GND #PWR03
+L power:GND #PWR010
 U 1 1 5E9ED404
 P 7150 4150
-F 0 "#PWR03" H 7150 3900 50  0001 C CNN
+F 0 "#PWR010" H 7150 3900 50  0001 C CNN
 F 1 "GND" H 7155 3977 50  0000 C CNN
 F 2 "" H 7150 4150 50  0001 C CNN
@@
 Wire Wire Line
 	8750 2650 8900 2650
+Text GLabel 5850 2600 2    50   Input ~ 0
+col0
+Text GLabel 5850 2700 2    50   Input ~ 0
+col1
+Text GLabel 5850 2800 2    50   Input ~ 0
+col2
+Text GLabel 5850 2900 2    50   Input ~ 0
+col3
+Text GLabel 5850 3000 2    50   Input ~ 0
+col4
+Text GLabel 5850 3100 2    50   Input ~ 0
+col5
+Text GLabel 5850 3200 2    50   Input ~ 0
+col6
+Text GLabel 5850 3300 2    50   Input ~ 0
+col7
+Text GLabel 5850 3500 2    50   Input ~ 0
+col8
+Text GLabel 5850 3600 2    50   Input ~ 0
+col9
+Text GLabel 5850 3800 2    50   Input ~ 0
+col10
+Text GLabel 5850 3900 2    50   Input ~ 0
+col11
+Text GLabel 5850 4000 2    50   Input ~ 0
+col12
+Text GLabel 5850 4100 2    50   Input ~ 0
+col13
+Text GLabel 5850 4200 2    50   Input ~ 0
+col14
+Text GLabel 5850 4300 2    50   Input ~ 0
+row0
+Text GLabel 5850 4400 2    50   Input ~ 0
+row1
+Text GLabel 5850 4500 2    50   Input ~ 0
+row2
+Text GLabel 5850 4800 2    50   Input ~ 0
+row3
+Text GLabel 5850 5000 2    50   Input ~ 0
+row4
+$Comp
+L Device:Rotary_Encoder_Switch SW2
+U 1 1 5E9943FC
+P 20550 9450
+F 0 "SW2" H 20550 9817 50  0000 C CNN
+F 1 "Rotary_Encoder_Switch" H 20550 9726 50  0000 C CNN
+F 2 "Keebio-Parts:RotaryEncoder_EC11" H 20400 9610 50  0001 C CNN
+F 3 "~" H 20550 9710 50  0001 C CNN
+	1    20550 9450
+	1    0    0    -1
+$EndComp
+$Comp
+L Device:Rotary_Encoder_Switch SW3
+U 1 1 5E997CC3
+P 20500 10450
+F 0 "SW3" H 20500 10817 50  0000 C CNN
+F 1 "Rotary_Encoder_Switch" H 20500 10726 50  0000 C CNN
+F 2 "Keebio-Parts:RotaryEncoder_EC11" H 20350 10610 50  0001 C CNN
+F 3 "~" H 20500 10710 50  0001 C CNN
+	1    20500 10450
+	1    0    0    -1
+$EndComp
+$Comp
+L Device:Rotary_Encoder_Switch SW4
+U 1 1 5E999039
+P 20500 11450
+F 0 "SW4" H 20500 11817 50  0000 C CNN
+F 1 "Rotary_Encoder_Switch" H 20500 11726 50  0000 C CNN
+F 2 "Keebio-Parts:RotaryEncoder_EC11" H 20350 11610 50  0001 C CNN
+F 3 "~" H 20500 11710 50  0001 C CNN
+	1    20500 11450
+	1    0    0    -1
+$EndComp
+Text GLabel 20850 9350 2    50   Input ~ 0
+0row
+Text GLabel 20850 9550 2    50   Input ~ 0
+0col
+Text GLabel 20800 10350 2    50   Input ~ 0
+1row
+Text GLabel 20800 10550 2    50   Input ~ 0
+1col
+Text GLabel 20800 11350 2    50   Input ~ 0
+2row
+Text GLabel 20800 11550 2    50   Input ~ 0
+2col
+Text GLabel 19100 11350 1    50   Input ~ 0
+2col
+Text GLabel 19100 10350 1    50   Input ~ 0
+1col
+Text GLabel 19100 9350 1    50   Input ~ 0
+0col
+Text GLabel 18900 9550 0    50   Input ~ 0
+0row
+Text GLabel 18900 10550 0    50   Input ~ 0
+1row
+Text GLabel 18900 11550 0    50   Input ~ 0
+2row
+$Comp
+L MX_Alps_Hybrid:MX-NoLED K_45
+U 1 1 5EA4E925
+P 18950 11400
+F 0 "K_45" H 18950 11633 60  0000 C CNN
+F 1 "KEYSW" H 18950 11300 60  0001 C CNN
+F 2 "MX_Only:MXOnly-1U-NoLED" H 18950 11400 60  0001 C CNN
+F 3 "" H 18950 11400 60  0000 C CNN
+	1    18950 11400
+	1    0    0    -1
+$EndComp
+$Comp
+L MX_Alps_Hybrid:MX-NoLED K_30
+U 1 1 5EA6F88E
+P 18950 10400
+F 0 "K_30" H 18950 10633 60  0000 C CNN
+F 1 "KEYSW" H 18950 10300 60  0001 C CNN
+F 2 "MX_Only:MXOnly-1U-NoLED" H 18950 10400 60  0001 C CNN
+F 3 "" H 18950 10400 60  0000 C CNN
+	1    18950 10400
+	1    0    0    -1
+$EndComp
+$Comp
+L MX_Alps_Hybrid:MX-NoLED K_15
+U 1 1 5EA90888
+P 18950 9400
+F 0 "K_15" H 18950 9633 60  0000 C CNN
+F 1 "KEYSW" H 18950 9300 60  0001 C CNN
+F 2 "MX_Only:MXOnly-1U-NoLED" H 18950 9400 60  0001 C CNN
+F 3 "" H 18950 9400 60  0000 C CNN
+	1    18950 9400
+	1    0    0    -1
+$EndComp
+Wire Wire Line
+	20250 9550 19750 9550
+Wire Wire Line
+	19750 10550 20200 10550
+Wire Wire Line
+	19750 11550 20200 11550
+$Comp
+L power:GND #PWR0101
+U 1 1 5EBE3CB7
+P 19850 11450
+F 0 "#PWR0101" H 19850 11200 50  0001 C CNN
+F 1 "GND" H 19855 11277 50  0000 C CNN
+F 2 "" H 19850 11450 50  0001 C CNN
+F 3 "" H 19850 11450 50  0001 C CNN
+	1    19850 11450
+	1    0    0    -1
+$EndComp
+$Comp
+L power:GND #PWR0102
+U 1 1 5EBE4F84
+P 19850 10450
+F 0 "#PWR0102" H 19850 10200 50  0001 C CNN
+F 1 "GND" H 19855 10277 50  0000 C CNN
+F 2 "" H 19850 10450 50  0001 C CNN
+F 3 "" H 19850 10450 50  0001 C CNN
+	1    19850 10450
+	1    0    0    -1
+$EndComp
+$Comp
+L power:GND #PWR0103
+U 1 1 5EBE5EB9
+P 19850 9450
+F 0 "#PWR0103" H 19850 9200 50  0001 C CNN
+F 1 "GND" H 19855 9277 50  0000 C CNN
+F 2 "" H 19850 9450 50  0001 C CNN
+F 3 "" H 19850 9450 50  0001 C CNN
+	1    19850 9450
+	1    0    0    -1
+$EndComp
+Wire Wire Line
+	19850 9450 20250 9450
+Wire Wire Line
+	19850 10450 20200 10450
+Wire Wire Line
+	19850 11450 20200 11450
+Text GLabel 19750 9350 1    50   Input ~ 0
+ENCB
+Text GLabel 20250 9350 0    50   Input ~ 0
+ENC0A
+Text GLabel 20200 10350 0    50   Input ~ 0
+ENC1A
+Text GLabel 20200 11350 0    50   Input ~ 0
+ENC2A
+Text GLabel 5850 5100 2    50   Input ~ 0
+ENCB
+Text GLabel 5850 5200 2    50   Input ~ 0
+ENC0A
+Text GLabel 5850 5300 2    50   Input ~ 0
+ENC1A
+Text GLabel 5850 5400 2    50   Input ~ 0
+ENC2A
+Connection ~ 19750 10550
+Wire Wire Line
+	19750 10550 19750 11550
+Wire Wire Line
+	19750 9350 19750 9550
+Connection ~ 19750 9550
+Wire Wire Line
+	19750 9550 19750 10550
 $EndSCHEMATC

Commit message: Assign Rows + Cols to pins
Connections:
- net 0col: now also U1.22 (PD5)
- net ENC0A: now also U1.25 (PD4)
- net ENC1A: now also U1.26 (PD6)
- net ENC2A: now also U1.27 (PD7)
- net ENCB: now also U1.28 (PB4)
- net col0: now also U1.41 (PF0)
- net col1: now also U1.40 (PF1)
- net col10: now also U1.18 (PD0)
- net col11: now also U1.19 (PD1)
- net col12: now also U1.20 (PD2)
- net col13: now also U1.21 (PD3)
- net col2: now also U1.39 (PF4)
- net col3: now also U1.32 (PC7)
- net col4: now also U1.31 (PC6)
- net col5: now also U1.30 (PB6)
- net col6: now also U1.29 (PB5)
- net col7: now also U1.9 (PB1)
- net col8: now also U1.10 (PB2)
- net col9: now also U1.11 (PB3)
- net row0: now also U1.8 (PB0)
- net row1: now also U1.12 (PB7)
- net row2: now also U1.38 (PF5)
- net row3: now also U1.37 (PF6)
- net row4: now also U1.36 (PF7)
Other:
- moved on the sheet: C1, C2, C3, C4, C5, D_1, D_10, D_11, D_12, D_13, D_14, D_15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
