File: Hardware/unnamed.kicad_pcb (KiCad board)
At the start: 2 copper layers, 15.2 x 6.3 mm, 156 parts, among them J1 USB2_C_Receptacle, SW1 SW_Push, SW2 Rotary_Encoder_Switch, SW3 Rotary_Encoder_Switch, SW4 Rotary_Encoder_Switch, U1 ATmega32U4-AU, U2 SRV05-4, Y1 16MHz

Commit message: Wire switch Matrix together
Parts:
- moved C1 99.3 mm to (270.4, 193.7)
- moved C2 99.3 mm to (274.4, 211.6)
- moved C3 99.3 mm to (280.1, 199.9)
- moved C5 99.3 mm to (265.2, 193.7)
- moved R1 99.3 mm to (279.3, 197.0)
- moved R6 99.3 mm to (266.3, 211.3)
- moved Y1 99.3 mm to (280.2, 202.8)
- moved C4 99.3 mm to (261.6, 206.2)
- moved R4 99.3 mm to (269.3, 189.6)
- moved R5 99.3 mm to (267.3, 189.6)
- moved U1 99.3 mm to (270.9, 202.5)
- moved SW1 86.2 mm to (277.2, 184.0), turned to 90 degrees
Routing:
- net row4: track 0.00 -> 337.0 mm
- net row2: track 0.00 -> 333.8 mm
- net row3: track 0.00 -> 311.3 mm
- net row1: track 0.00 -> 294.6 mm
- net row0: track 0.00 -> 290.6 mm

Commit message: Wire MCU + GND fill
Parts:
- moved F1 40.3 mm to (276.4, 154.5)
- moved J1 40.3 mm to (276.3, 143.3)
- moved R2 40.3 mm to (270.0, 153.8)
- moved R3 40.3 mm to (282.7, 153.8)
- moved U2 40.3 mm to (276.3, 157.6)
- moved SW1 18.9 mm to (289.8, 198.1), turned to 10 degrees
- moved R4 0.55 mm to (269.9, 189.6)
- moved R5 0.55 mm to (267.9, 189.6)
Connections:
- U1 pad 10: Net-(U1-Pad10) -> col8
- U1 pad 11: Net-(U1-Pad11) -> col7
- U1 pad 12: Net-(U1-Pad12) -> row1
- U1 pad 18: Net-(U1-Pad18) -> 0col
- U1 pad 19: Net-(U1-Pad19) -> col13
- U1 pad 20: Net-(U1-Pad20) -> col12
- U1 pad 21: Net-(U1-Pad21) -> col11
- U1 pad 22: Net-(U1-Pad22) -> col10
- U1 pad 25: Net-(U1-Pad25) -> ENC0A
- U1 pad 26: Net-(U1-Pad26) -> ENC1A
- U1 pad 27: Net-(U1-Pad27) -> ENC2A
- U1 pad 28: Net-(U1-Pad28) -> ENCB
- U1 pad 29: Net-(U1-Pad29) -> col6
- U1 pad 30: Net-(U1-Pad30) -> row4
- U1 pad 31: Net-(U1-Pad31) -> row3
- U1 pad 32: Net-(U1-Pad32) -> col5
- U1 pad 36: Net-(U1-Pad36) -> row2
- U1 pad 37: Net-(U1-Pad37) -> col4
- U1 pad 38: Net-(U1-Pad38) -> col3
- U1 pad 39: Net-(U1-Pad39) -> col2
- U1 pad 40: Net-(U1-Pad40) -> col1
- U1 pad 41: Net-(U1-Pad41) -> col0
- U1 pad 8: Net-(U1-Pad8) -> row0
- U1 pad 9: Net-(U1-Pad9) -> col9
Routing:
- net ENCB: track 0.00 -> 257.7 mm
- net ENC0A: track 0.00 -> 231.2 mm, vias 0 -> 1
- net ENC1A: track 0.00 -> 217.4 mm, vias 0 -> 1
- net ENC2A: track 0.00 -> 205.8 mm
- net 0col: track 94.2 -> 294.2 mm, vias 0 -> 1
- net col13: track 95.2 -> 253.6 mm, vias 0 -> 1
- net col12: track 94.8 -> 230.2 mm, vias 0 -> 1
- net col0: track 87.9 -> 219.7 mm, vias 0 -> 1
- net col11: track 92.6 -> 207.6 mm, vias 0 -> 1
- net col1: track 90.0 -> 198.0 mm, vias 0 -> 1
- net +5V: track 0.00 -> 100.2 mm, vias 0 -> 7
- net col10: track 92.9 -> 189.8 mm, vias 0 -> 1
- net col2: track 87.6 -> 171.1 mm, vias 0 -> 1
- net col9: track 89.0 -> 172.2 mm
- net row0: track 290.6 -> 361.3 mm, vias 0 -> 2
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- added copper zone on B.Cu, net GND
- added copper zone on F.Cu, net GND
Other:
- board size 15.2 x 6.3 mm -> 361 x 120.8 mm
