File: Hardware/Rev 0.2 RGB/trifecta.kicad_pcb (KiCad board)
At the start: 2 copper layers, 361 x 120.8 mm, 261 parts, among them J1 USB2_C_Receptacle, SW1 SW_Push, SW2 Rotary_Encoder_Switch, SW3 Rotary_Encoder_Switch, SW4 Rotary_Encoder_Switch, U1 ATmega32U4-AU, U2 SRV05-4, Y1 16MHz

Commit message: Add Step of PCB
Parts:
- moved C69 167.7 mm to (336.8, 118.7)
- moved C70 167.7 mm to (355.9, 118.7)
- moved D_12 167.7 mm to (273.7, 32.5)
- moved D_26 167.7 mm to (269.0, 52.5)
- moved D_29 167.7 mm to (330.9, 52.5)
- moved D_67 167.7 mm to (299.9, 109.6)
- moved K_13 167.7 mm to (284.5, 29.6)
- moved K_15 167.7 mm to (351.2, 29.6)
- moved K_26 167.7 mm to (260.7, 48.6)
- moved K_56 167.7 mm to (260.7, 86.7)
- moved K_70 167.7 mm to (355.9, 110.5)
- moved LED26 167.7 mm to (260.6, 54.0)
- moved LED57 167.7 mm to (279.7, 92.1)
- moved LED59 167.7 mm to (336.8, 96.9)
- moved LED68 167.7 mm to (317.7, 115.9)
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
Commit message: PCB Final
Parts:
- removed the G*** at (171.2, 120.9)
- removed the K_31 at (32.5, 67.7)
- added D_16: D, kbd:D3_SMD_v2, B.Cu at (438.8, 162.2)
- added G***: LOGO, graphics:image1, B.Cu at (278.7, 250.9)
- added K_14: KEYSW, MX_Only:MXOnly-1U-NoLED, F.Cu at (411.1, 158.3)
- added K_16: KEYSW, MX_Only:MXOnly-1U-NoLED, F.Cu at (430.0, 158.3)
- added K_32: KEYSW, MX_Only:MXOnly-1.75U-NoLED, F.Cu at (139.9, 196.4)
- D_1, D_10, D_11, D_12, D_13, D_2, D_3, D_4, D_5, D_6, D_7, D_8, D_9: footprint kbd:D_SOD-123_copy -> kbd:D3_SMD_v2
- D_15: renamed from D_14; footprint kbd:D_SOD-123_copy -> kbd:D3_SMD_v2
- D_17: renamed from D_16; footprint kbd:D_SOD-123_copy -> kbd:D3_SMD_v2
- D_18: renamed from D_17; footprint kbd:D_SOD-123_copy -> kbd:D3_SMD_v2
- D_19: renamed from D_18; footprint kbd:D_SOD-123_copy -> kbd:D3_SMD_v2
- D_20: renamed from D_19; footprint kbd:D_SOD-123_copy -> kbd:D3_SMD_v2
- D_21: renamed from D_20; footprint kbd:D_SOD-123_copy -> kbd:D3_SMD_v2
- D_22: renamed from D_21; footprint kbd:D_SOD-123_copy -> kbd:D3_SMD_v2
- D_23: renamed from D_22; footprint kbd:D_SOD-123_copy -> kbd:D3_SMD_v2
- D_24: renamed from D_23; footprint kbd:D_SOD-123_copy -> kbd:D3_SMD_v2
- D_25: renamed from D_24; footprint kbd:D_SOD-123_copy -> kbd:D3_SMD_v2
- D_26: renamed from D_25; footprint kbd:D_SOD-123_copy -> kbd:D3_SMD_v2
- D_27: renamed from D_26; footprint kbd:D_SOD-123_copy -> kbd:D3_SMD_v2
- D_28: renamed from D_27; footprint kbd:D_SOD-123_copy -> kbd:D3_SMD_v2
- D_29: renamed from D_28; footprint kbd:D_SOD-123_copy -> kbd:D3_SMD_v2
- D_30: renamed from D_29; footprint kbd:D_SOD-123_copy -> kbd:D3_SMD_v2
- D_31: renamed from D_15; footprint kbd:D_SOD-123_copy -> kbd:D3_SMD_v2
- D_33: renamed from D_31; footprint kbd:D_SOD-123_copy -> kbd:D3_SMD_v2
- D_34: renamed from D_33; footprint kbd:D_SOD-123_copy -> kbd:D3_SMD_v2
- D_35: renamed from D_34; footprint kbd:D_SOD-123_copy -> kbd:D3_SMD_v2
- D_36: renamed from D_35; footprint kbd:D_SOD-123_copy -> kbd:D3_SMD_v2
- D_37: renamed from D_36; footprint kbd:D_SOD-123_copy -> kbd:D3_SMD_v2
- D_38: renamed from D_37; footprint kbd:D_SOD-123_copy -> kbd:D3_SMD_v2
- D_39: renamed from D_38; footprint kbd:D_SOD-123_copy -> kbd:D3_SMD_v2
- D_40: renamed from D_39; footprint kbd:D_SOD-123_copy -> kbd:D3_SMD_v2
- D_41: renamed from D_40; footprint kbd:D_SOD-123_copy -> kbd:D3_SMD_v2
- D_42: renamed from D_41; footprint kbd:D_SOD-123_copy -> kbd:D3_SMD_v2
- D_43: renamed from D_42; footprint kbd:D_SOD-123_copy -> kbd:D3_SMD_v2
- D_44: renamed from D_43; footprint kbd:D_SOD-123_copy -> kbd:D3_SMD_v2
- D_45: renamed from D_44; footprint kbd:D_SOD-123_copy -> kbd:D3_SMD_v2
- D_46: renamed from D_30; footprint kbd:D_SOD-123_copy -> kbd:D3_SMD_v2
- D_47: renamed from D_46; footprint kbd:D_SOD-123_copy -> kbd:D3_SMD_v2
- D_48: renamed from D_47; footprint kbd:D_SOD-123_copy -> kbd:D3_SMD_v2
- D_49: renamed from D_48; footprint kbd:D_SOD-123_copy -> kbd:D3_SMD_v2
- D_50: renamed from D_49; footprint kbd:D_SOD-123_copy -> kbd:D3_SMD_v2
- D_51: renamed from D_50; footprint kbd:D_SOD-123_copy -> kbd:D3_SMD_v2
- D_52: renamed from D_51; footprint kbd:D_SOD-123_copy -> kbd:D3_SMD_v2
- D_53: renamed from D_52; footprint kbd:D_SOD-123_copy -> kbd:D3_SMD_v2
- D_54: renamed from D_53; footprint kbd:D_SOD-123_copy -> kbd:D3_SMD_v2
- D_55: renamed from D_54; footprint kbd:D_SOD-123_copy -> kbd:D3_SMD_v2
- D_56: renamed from D_55; footprint kbd:D_SOD-123_copy -> kbd:D3_SMD_v2
- D_57: renamed from D_56; footprint kbd:D_SOD-123_copy -> kbd:D3_SMD_v2
- D_58: renamed from D_57; footprint kbd:D_SOD-123_copy -> kbd:D3_SMD_v2
- D_59: renamed from D_58; footprint kbd:D_SOD-123_copy -> kbd:D3_SMD_v2
- D_60: renamed from D_59; footprint kbd:D_SOD-123_copy -> kbd:D3_SMD_v2
- D_61: renamed from D_45; footprint kbd:D_SOD-123_copy -> kbd:D3_SMD_v2
- D_62: renamed from D_60; footprint kbd:D_SOD-123_copy -> kbd:D3_SMD_v2
- D_63: renamed from D_61; footprint kbd:D_SOD-123_copy -> kbd:D3_SMD_v2
- D_64: renamed from D_62; footprint kbd:D_SOD-123_copy -> kbd:D3_SMD_v2
- D_65: renamed from D_63; footprint kbd:D_SOD-123_copy -> kbd:D3_SMD_v2
- D_66: renamed from D_64; footprint kbd:D_SOD-123_copy -> kbd:D3_SMD_v2
- D_67: renamed from D_65; footprint kbd:D_SOD-123_copy -> kbd:D3_SMD_v2
- D_68: renamed from D_66; footprint kbd:D_SOD-123_copy -> kbd:D3_SMD_v2
- D_69: renamed from D_67; footprint kbd:D_SOD-123_copy -> kbd:D3_SMD_v2
- D_70: renamed from D_68; footprint kbd:D_SOD-123_copy -> kbd:D3_SMD_v2
- D_71: renamed from D_69; footprint kbd:D_SOD-123_copy -> kbd:D3_SMD_v2
- D_72: renamed from D_70; footprint kbd:D_SOD-123_copy -> kbd:D3_SMD_v2
- K_15: renamed from K_14; footprint MX_Only:MXOnly-2U-ReversedStabilizers-NoLED -> MX_Only:MXOnly-2U-NoLED
- K_30: renamed from K_29; footprint MX_Only:MXOnly-1.5U-NoLED -> MX_Only:MXOnly-1U-NoLED
- U1: footprint Package_QFP:TQFP-44_10x10mm_P0.8mm -> Keebio-Parts:ATMEGA32U4-AU
- moved C71 167.7 mm to (444.2, 247.4)
- moved C72 167.7 mm to (463.3, 247.4)
- moved D_12 167.7 mm to (381.1, 161.2)
- moved D_27 167.7 mm to (376.4, 181.2)
- moved D_30 167.7 mm to (438.3, 181.2)
- moved D_69 167.7 mm to (407.4, 238.4)
- moved K_13 167.7 mm to (391.9, 158.3)
- moved K_27 167.7 mm to (368.1, 177.4)
- moved K_31 167.7 mm to (458.6, 158.3)
- moved K_57 167.7 mm to (368.1, 215.5)
- moved K_72 167.7 mm to (463.3, 239.3)
- moved LED27 167.7 mm to (368.0, 182.7)
- moved LED58 167.7 mm to (387.2, 220.8)
- moved LED60 167.7 mm to (444.2, 225.6)
- moved LED70 167.7 mm to (425.1, 244.7)
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- renumbered C14 to C15, C15 to C16, C17 to C18, C19 to C20, C21 to C22, C23 to C24, C25 to C26, C27 to C28, C29 to C30, C33 to C34, C35 to C36, C37 to C38, C39 to C40, C41 to C42, C43 to C44, C44 to C45, C47 to C48, C49 to C50, C51 to C52, C53 to C54, C55 to C56, C57 to C58, C59 to C60, C61 to C63, C64 to C66, C65 to C67, C67 to C69, C69 to C71, C70 to C72, K_16 to K_17, K_17 to K_18, K_18 to K_19, K_19 to K_20, K_20 to K_21, K_21 to K_22, K_22 to K_23, K_23 to K_24, K_24 to K_25, K_25 to K_26, K_26 to K_27, K_27 to K_28, K_28 to K_29, K_15 to K_31, K_32 to K_33, K_33 to K_34, K_34 to K_35, K_35 to K_36, K_36 to K_37, K_37 to K_38, K_38 to K_39, K_39 to K_40, K_40 to K_41, K_41 to K_42, K_42 to K_43, K_43 to K_44, K_44 to K_45, K_30 to K_46, K_46 to K_47, K_47 to K_48, K_48 to K_49, K_49 to K_50, K_50 to K_51, K_51 to K_52, K_52 to K_53, K_53 to K_54, K_54 to K_55, K_55 to K_56, K_56 to K_57, K_57 to K_58, K_58 to K_59, K_59 to K_60, K_45 to K_61, K_60 to K_62, K_61 to K_63, K_62 to K_64, K_63 to K_65, K_64 to K_66, K_65 to K_67, K_66 to K_68, K_67 to K_69, K_68 to K_70, K_69 to K_71, K_70 to K_72, LED14 to LED15, LED16 to LED17, LED17 to LED18, LED18 to LED19, LED19 to LED20, LED20 to LED21, LED21 to LED22, LED22 to LED23, LED23 to LED24, LED24 to LED25, LED25 to LED26, LED26 to LED27, LED27 to LED28, LED28 to LED29, LED29 to LED30, LED32 to LED33, LED33 to LED34, LED34 to LED35, LED35 to LED36, LED36 to LED37, LED37 to LED38, LED38 to LED39, LED39 to LED40, LED40 to LED41, LED41 to LED42, LED42 to LED43, LED43 to LED44, LED44 to LED45, LED46 to LED47, LED47 to LED48, LED48 to LED49, LED49 to LED50, LED50 to LED51, LED51 to LED52, LED52 to LED53, LED53 to LED54, LED54 to LED55, LED55 to LED56, LED56 to LED57, LED57 to LED58, LED58 to LED59, LED59 to LED60, LED60 to LED62, LED61 to LED63, LED62 to LED64, LED63 to LED65, LED64 to LED66, LED65 to LED67, LED66 to LED68, LED67 to LED69, LED68 to LED70, LED69 to LED71, LED70 to LED72
Connections:
- D_31 pad 1: row0 -> row1
- D_46 pad 1: row1 -> row2
- D_61 pad 1: row2 -> row3
Routing:
- net GND: track 2269.9 -> 2411.7 mm, vias 96 -> 111
- net 0col: track 297.2 -> 329.5 mm
- net row3: track 347.1 -> 378.0 mm
- net row0: track 368.0 -> 340.5 mm
- net Net-(D_16-Pad2): track 0.00 -> 11.7 mm
- net col13: track 267.1 -> 277.7 mm
- net Net-(D_15-Pad2): track 21.2 -> 31.0 mm
- net row2: track 358.9 -> 368.1 mm
- net row1: track 355.7 -> 362.8 mm
- net +5V: track 1913.8 -> 1917.0 mm
- net Net-(D_30-Pad2): track 13.0 -> 11.7 mm
