File: Hardware/Rev 0.2 RGB/trifecta.kicad_pcb (KiCad board)
At the start: 2 copper layers, 361 x 120.8 mm, 264 parts, among them J1 USB2_C_Receptacle, SW1 SW_Push, SW2 Rotary_Encoder_Switch, SW3 Rotary_Encoder_Switch, SW4 Rotary_Encoder_Switch, U1 ATmega32U4-AU, U2 SRV05-4, Y1 16MHz

Commit message: Add new laser cut DXF files
Parts:
- moved D_24 200.8 mm to (180.9, 39.1)
- moved K_66 200.8 mm to (175.0, 94.7)
- moved LED58 200.8 mm to (252.5, 72.0)
- moved C1 200.8 mm to (135.7, 44.8)
- moved C10 200.8 mm to (198.3, 21.3)
- moved C11 200.8 mm to (145.4, 51.0)
- moved C12 200.8 mm to (237.9, 17.5)
- moved C13 200.8 mm to (127.0, 57.3)
- moved C15 200.8 mm to (285.7, 17.5)
- moved C16 200.8 mm to (130.5, 44.8)
- moved C18 200.8 mm to (33.3, 36.5)
- moved C2 200.8 mm to (28.6, 17.6)
- moved C20 200.8 mm to (74.6, 40.0)
- moved C22 200.8 mm to (112.1, 46.6)
- moved C24 200.8 mm to (173.6, 45.0)
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
Commit message: Update Gerbers
Routing:
- net GND: vias 111 -> 135
