File: Hardware/Rev 0.2 RGB/trifecta.sch (KiCad schematic (older format))
At the start: 260 parts, among them J1 USB2_C_Receptacle, SW1 SW_Push, SW2 Rotary_Encoder_Switch, SW3 Rotary_Encoder_Switch, SW4 Rotary_Encoder_Switch, U1 ATmega32U4-AU, U2 SRV05-4, Y1 16MHz

Commit message: Names of PCBs
Parts:
- C1, C11, C13, C15, C9: symbol unnamed-rescue:C_Small-Device -> trifecta-rescue:C_Small-Device-unnamed-rescue
- C10, C12, C14, C17, C19, C2, C21, C23, C25, C27, C29, C33, C35, C37, C39, C4, C41, C43, C44, C47, C49, C51, C53, C55, C57, C59, C6, C61, C64, C65, C67, C69, C70, C8: symbol unnamed-rescue:C_Small-device -> trifecta-rescue:C_Small-device-unnamed-rescue
- D_1, D_10, D_11, D_12, D_13, D_14, D_15, D_16, D_17, D_18, D_19, D_2, D_20, D_21, D_22, D_23, D_24, D_25, D_26, D_27, D_28, D_29, D_3, D_30, D_31, D_33, D_34, D_35, D_36, D_37, D_38, D_39, D_4, D_40, D_41, D_42, D_43, D_44, D_45, D_46, D_47, D_48, D_49, D_5, D_50, D_51, D_52, D_53, D_54, D_55, D_56, D_57, D_58, D_59, D_6, D_60, D_61, D_62, D_63, D_64, D_65, D_66, D_67, D_68, D_69, D_7, D_70, D_8, D_9: symbol unnamed-rescue:D_Small-Device -> trifecta-rescue:D_Small-Device-unnamed-rescue
- F1: symbol unnamed-rescue:Polyfuse_Small-Device -> trifecta-rescue:Polyfuse_Small-Device-unnamed-rescue
- K_15, K_30, K_45: renamed from K_?; footprint MX_Only:MXOnly-2.25U-ReversedStabilizers-NoLED -> MX_Only:MXOnly-1U-NoLED
- LED1, LED10, LED11, LED12, LED13, LED14, LED16, LED17, LED18, LED19, LED2, LED20, LED21, LED22, LED23, LED24, LED25, LED26, LED27, LED28, LED29, LED3, LED32, LED33, LED34, LED35, LED36, LED37, LED38, LED39, LED4, LED40, LED41, LED42, LED43, LED44, LED46, LED47, LED48, LED49, LED5, LED50, LED51, LED52, LED53, LED54, LED55, LED56, LED57, LED58, LED59, LED6, LED60, LED61, LED62, LED63, LED64, LED65, LED66, LED67, LED68, LED69, LED7, LED70, LED8, LED9: symbol unnamed-rescue:WS2812B-Worldsemi -> trifecta-rescue:WS2812B-Worldsemi-unnamed-rescue
- R1, R2, R3, R4, R5, R6: symbol unnamed-rescue:R_Small-Device -> trifecta-rescue:R_Small-Device-unnamed-rescue
- R7: symbol unnamed-rescue:R_Small-device -> trifecta-rescue:R_Small-device-unnamed-rescue
- SW1: symbol unnamed-rescue:SW_Push-Switch -> trifecta-rescue:SW_Push-Switch-unnamed-rescue
- SW2, SW3, SW4: symbol unnamed-rescue:Rotary_Encoder_Switch-Device -> trifecta-rescue:Rotary_Encoder_Switch-Device-unnamed-rescue
- U1: symbol unnamed-rescue:ATmega32U4-AU-MCU_Microchip_ATmega -> trifecta-rescue:ATmega32U4-AU-MCU_Microchip_ATmega-unnamed-rescue
- U2: symbol unnamed-rescue:SRV05-4-Power_Protection -> trifecta-rescue:SRV05-4-Power_Protection-unnamed-rescue
- Y1: symbol unnamed-rescue:Resonator_Small-Device -> trifecta-rescue:Resonator_Small-Device-unnamed-rescue

Commit message: PCB Final
Parts:
- removed K_31: KEYSW, MX_Only:MXOnly-1.25U-NoLED, symbol MX_Alps_Hybrid:MX-NoLED
- added D_16: D, kbd:D3_SMD_v2, symbol trifecta-rescue:D_Small-Device-unnamed-rescue
- added K_14, K_16: KEYSW, MX_Only:MXOnly-1U-NoLED, symbol MX_Alps_Hybrid:MX-NoLED
- added K_32: KEYSW, MX_Only:MXOnly-1.75U-NoLED, symbol MX_Alps_Hybrid:MX-NoLED
- D_1, D_10, D_11, D_12, D_13, D_2, D_3, D_4, D_5, D_6, D_7, D_8, D_9: footprint kbd:D_SOD-123_copy -> kbd:D3_SMD_v2
- D_15: renamed from D_14; footprint kbd:D_SOD-123_copy -> kbd:D3_SMD_v2
- D_17: renamed from D_16; footprint kbd:D_SOD-123_copy -> kbd:D3_SMD_v2
- D_18: renamed from D_17; footprint kbd:D_SOD-123_copy -> kbd:D3_SMD_v2
- D_19: renamed from D_18; footprint kbd:D_SOD-123_copy -> kbd:D3_SMD_v2
- D_20: renamed from D_19; footprint kbd:D_SOD-123_copy -> kbd:D3_SMD_v2
- D_21: renamed from D_20; footprint kbd:D_SOD-123_copy -> kbd:D3_SMD_v2
- D_22: renamed from D_21; footprint kbd:D_SOD-123_copy -> kbd:D3_SMD_v2
- D_23: renamed from D_22; footprint kbd:D_SOD-123_copy -> kbd:D3_SMD_v2
- D_24: renamed from D_23; footprint kbd:D_SOD-123_copy -> kbd:D3_SMD_v2
- D_25: renamed from D_24; footprint kbd:D_SOD-123_copy -> kbd:D3_SMD_v2
- D_26: renamed from D_25; footprint kbd:D_SOD-123_copy -> kbd:D3_SMD_v2
- D_27: renamed from D_26; footprint kbd:D_SOD-123_copy -> kbd:D3_SMD_v2
- D_28: renamed from D_27; footprint kbd:D_SOD-123_copy -> kbd:D3_SMD_v2
- D_29: renamed from D_28; footprint kbd:D_SOD-123_copy -> kbd:D3_SMD_v2
- D_30: renamed from D_29; footprint kbd:D_SOD-123_copy -> kbd:D3_SMD_v2
- D_31: renamed from D_15; footprint kbd:D_SOD-123_copy -> kbd:D3_SMD_v2
- D_33: renamed from D_31; footprint kbd:D_SOD-123_copy -> kbd:D3_SMD_v2
- D_34: renamed from D_33; footprint kbd:D_SOD-123_copy -> kbd:D3_SMD_v2
- D_35: renamed from D_34; footprint kbd:D_SOD-123_copy -> kbd:D3_SMD_v2
- D_36: renamed from D_35; footprint kbd:D_SOD-123_copy -> kbd:D3_SMD_v2
- D_37: renamed from D_36; footprint kbd:D_SOD-123_copy -> kbd:D3_SMD_v2
- D_38: renamed from D_37; footprint kbd:D_SOD-123_copy -> kbd:D3_SMD_v2
- D_39: renamed from D_38; footprint kbd:D_SOD-123_copy -> kbd:D3_SMD_v2
- D_40: renamed from D_39; footprint kbd:D_SOD-123_copy -> kbd:D3_SMD_v2
- D_41: renamed from D_40; footprint kbd:D_SOD-123_copy -> kbd:D3_SMD_v2
- D_42: renamed from D_41; footprint kbd:D_SOD-123_copy -> kbd:D3_SMD_v2
- D_43: renamed from D_42; footprint kbd:D_SOD-123_copy -> kbd:D3_SMD_v2
- D_44: renamed from D_43; footprint kbd:D_SOD-123_copy -> kbd:D3_SMD_v2
- D_45: renamed from D_44; footprint kbd:D_SOD-123_copy -> kbd:D3_SMD_v2
- D_46: renamed from D_30; footprint kbd:D_SOD-123_copy -> kbd:D3_SMD_v2
- D_47: renamed from D_46; footprint kbd:D_SOD-123_copy -> kbd:D3_SMD_v2
- D_48: renamed from D_47; footprint kbd:D_SOD-123_copy -> kbd:D3_SMD_v2
- D_49: renamed from D_48; footprint kbd:D_SOD-123_copy -> kbd:D3_SMD_v2
- D_50: renamed from D_49; footprint kbd:D_SOD-123_copy -> kbd:D3_SMD_v2
- D_51: renamed from D_50; footprint kbd:D_SOD-123_copy -> kbd:D3_SMD_v2
- D_52: renamed from D_51; footprint kbd:D_SOD-123_copy -> kbd:D3_SMD_v2
- D_53: renamed from D_52; footprint kbd:D_SOD-123_copy -> kbd:D3_SMD_v2
- D_54: renamed from D_53; footprint kbd:D_SOD-123_copy -> kbd:D3_SMD_v2
- D_55: renamed from D_54; footprint kbd:D_SOD-123_copy -> kbd:D3_SMD_v2
- D_56: renamed from D_55; footprint kbd:D_SOD-123_copy -> kbd:D3_SMD_v2
- D_57: renamed from D_56; footprint kbd:D_SOD-123_copy -> kbd:D3_SMD_v2
- D_58: renamed from D_57; footprint kbd:D_SOD-123_copy -> kbd:D3_SMD_v2
- D_59: renamed from D_58; footprint kbd:D_SOD-123_copy -> kbd:D3_SMD_v2
- D_60: renamed from D_59; footprint kbd:D_SOD-123_copy -> kbd:D3_SMD_v2
- D_61: renamed from D_45; footprint kbd:D_SOD-123_copy -> kbd:D3_SMD_v2
- D_62: renamed from D_60; footprint kbd:D_SOD-123_copy -> kbd:D3_SMD_v2
- D_63: renamed from D_61; footprint kbd:D_SOD-123_copy -> kbd:D3_SMD_v2
- D_64: renamed from D_62; footprint kbd:D_SOD-123_copy -> kbd:D3_SMD_v2
- D_65: renamed from D_63; footprint kbd:D_SOD-123_copy -> kbd:D3_SMD_v2
- D_66: renamed from D_64; footprint kbd:D_SOD-123_copy -> kbd:D3_SMD_v2
- D_67: renamed from D_65; footprint kbd:D_SOD-123_copy -> kbd:D3_SMD_v2
- D_68: renamed from D_66; footprint kbd:D_SOD-123_copy -> kbd:D3_SMD_v2
- D_69: renamed from D_67; footprint kbd:D_SOD-123_copy -> kbd:D3_SMD_v2
- D_70: renamed from D_68; footprint kbd:D_SOD-123_copy -> kbd:D3_SMD_v2
- D_71: renamed from D_69; footprint kbd:D_SOD-123_copy -> kbd:D3_SMD_v2
- D_72: renamed from D_70; footprint kbd:D_SOD-123_copy -> kbd:D3_SMD_v2
- K_15: renamed from K_14; footprint MX_Only:MXOnly-2U-ReversedStabilizers-NoLED -> MX_Only:MXOnly-2U-NoLED
- K_30: renamed from K_29; footprint MX_Only:MXOnly-1.5U-NoLED -> MX_Only:MXOnly-1U-NoLED
- U1: footprint Package_QFP:TQFP-44_10x10mm_P0.8mm -> Keebio-Parts:ATMEGA32U4-AU
- renumbered C14 to C15, C15 to C16, C17 to C18, C19 to C20, C21 to C22, C23 to C24, C25 to C26, C27 to C28, C29 to C30, C33 to C34, C35 to C36, C37 to C38, C39 to C40, C41 to C42, C43 to C44, C44 to C45, C47 to C48, C49 to C50, C51 to C52, C53 to C54, C55 to C56, C57 to C58, C59 to C60, C61 to C63, C64 to C66, C65 to C67, C67 to C69, C69 to C71, C70 to C72, K_16 to K_17, K_17 to K_18, K_18 to K_19, K_19 to K_20, K_20 to K_21, K_21 to K_22, K_22 to K_23, K_23 to K_24, K_24 to K_25, K_25 to K_26, K_26 to K_27, K_27 to K_28, K_28 to K_29, K_15 to K_31, K_32 to K_33, K_33 to K_34, K_34 to K_35, K_35 to K_36, K_36 to K_37, K_37 to K_38, K_38 to K_39, K_39 to K_40, K_40 to K_41, K_41 to K_42, K_42 to K_43, K_43 to K_44, K_44 to K_45, K_30 to K_46, K_46 to K_47, K_47 to K_48, K_48 to K_49, K_49 to K_50, K_50 to K_51, K_51 to K_52, K_52 to K_53, K_53 to K_54, K_54 to K_55, K_55 to K_56, K_56 to K_57, K_57 to K_58, K_58 to K_59, K_59 to K_60, K_45 to K_61, K_60 to K_62, K_61 to K_63, K_62 to K_64, K_63 to K_65, K_64 to K_66, K_65 to K_67, K_66 to K_68, K_67 to K_69, K_68 to K_70, K_69 to K_71, K_70 to K_72, LED14 to LED15, LED16 to LED17, LED17 to LED18, LED18 to LED19, LED19 to LED20, LED20 to LED21, LED21 to LED22, LED22 to LED23, LED23 to LED24, LED24 to LED25, LED25 to LED26, LED26 to LED27, LED27 to LED28, LED28 to LED29, LED29 to LED30, LED32 to LED33, LED33 to LED34, LED34 to LED35, LED35 to LED36, LED36 to LED37, LED37 to LED38, LED38 to LED39, LED39 to LED40, LED40 to LED41, LED41 to LED42, LED42 to LED43, LED43 to LED44, LED44 to LED45, LED46 to LED47, LED47 to LED48, LED48 to LED49, LED49 to LED50, LED50 to LED51, LED51 to LED52, LED52 to LED53, LED53 to LED54, LED54 to LED55, LED55 to LED56, LED56 to LED57, LED57 to LED58, LED58 to LED59, LED59 to LED60, LED60 to LED62, LED61 to LED63, LED62 to LED64, LED63 to LED65, LED64 to LED66, LED65 to LED67, LED66 to LED68, LED67 to LED69, LED68 to LED70, LED69 to LED71, LED70 to LED72
Connections:
- net 0col: now also K_16.1 (COL)
- net col0: now also K_32.1 (COL)
- net col13: now also K_14.1 (COL)
- net row0: now also D_16.1 (K); no longer D_31.1 (K)
- net row1: now also D_31.1 (K); no longer D_46.1 (K)
- net row2: now also D_46.1 (K); no longer D_61.1 (K)
- net row3: now also D_61.1 (K)
- net at D_33.2 (A), K_33.2 (ROW): now also K_32.2 (ROW)
- net at D_15.2 (A), K_15.2 (ROW): now also K_14.2 (ROW)
- new net: D_16.2 (A), K_16.2 (ROW)
Other:
- moved on the sheet: D_1, D_10, D_11, D_12, D_13, D_15, D_17, D_18, D_19, D_2, D_20, D_21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
