File: Hardware/Rev 0.5 RGB/trifecta.kicad_pcb (KiCad board)
At the start: 2 copper layers, 361 x 120.8 mm, 285 parts, among them J1 USB2_C_Receptacle, SW1 SW_Push, SW2 Rotary_Encoder_Switch, SW3 Rotary_Encoder_Switch, SW4 Rotary_Encoder_Switch, U1 ATmega32U4-AU, U2 SRV05-4, Y1 16MHz

Commit message: LED Update
Parts:
- moved ULED11 6.53 mm to (178.6, 6.20), turned to 180 degrees
- moved ULED10 6.29 mm to (113.6, 4.70), turned to 180 degrees
- moved ULED13 5.01 mm to (255.6, 0.81), turned to 180 degrees
- moved ULED14 4.89 mm to (310.6, 24.5), turned to 180 degrees
- moved ULED12 4.89 mm to (219.7, 24.3), turned to 180 degrees
- moved ULED8 4.76 mm to (45.3, 21.9), turned to 180 degrees
- moved ULED9 4.55 mm to (87.0, 26.7), turned to 180 degrees
- moved ULED4 0.71 mm to (224.8, 84.2)
- moved ULED6 0.61 mm to (47.0, 85.2)
- moved ULED3 0.41 mm to (278.1, 83.5)
- moved ULED5 0.29 mm to (138.6, 109.9)
- moved ULED1 0.28 mm to (339.6, 6.45)
- moved ULED7 0.21 mm to (-5.28, 7.98)
- moved ULED2 0.13 mm to (333.7, 74.9)
- turned C73 to 180 degrees
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
Commit message: 08/07
Parts:
- moved ULED5 5.02 mm to (138.6, 104.9), turned to 0 degrees
- moved ULED3 4.98 mm to (278.1, 78.5), turned to 0 degrees
- moved ULED12 0.94 mm to (220.4, 23.7)
- moved C75 0.37 mm to (278.1, 83.6), turned to 0 degrees
- turned C77 to 0 degrees
Connections:
- ULED6 pad 4: Net-(ULED6-Pad4) -> Net-(ULED5-Pad2)
- ULED9 pad 4: Net-(ULED9-Pad4) -> Net-(ULED8-Pad2)
Routing:
- net +5V: track 1924.5 -> 2370.5 mm, vias 78 -> 91
- net GND: track 2445.2 -> 2707.4 mm, vias 129 -> 141
- net Net-(ULED6-Pad2): track 0.00 -> 135.9 mm, vias 0 -> 1
- net Net-(ULED5-Pad2): track 0.00 -> 118.6 mm, vias 0 -> 2
- net Net-(ULED4-Pad2): track 0.00 -> 112.8 mm, vias 0 -> 2
- net Net-(ULED1-Pad2): track 0.00 -> 77.6 mm, vias 0 -> 2
- net Net-(ULED10-Pad2): track 0.00 -> 73.0 mm, vias 0 -> 4
- net Net-(ULED13-Pad2): track 0.00 -> 70.5 mm, vias 0 -> 2
- net Net-(ULED2-Pad2): track 0.00 -> 70.0 mm, vias 0 -> 2
- net Net-(ULED3-Pad2): track 0.00 -> 56.8 mm
- net Net-(ULED7-Pad2): track 0.00 -> 56.3 mm, vias 0 -> 2
- net Net-(ULED11-Pad2): track 0.00 -> 50.8 mm, vias 0 -> 4
- net Net-(ULED12-Pad2): track 0.00 -> 49.8 mm, vias 0 -> 2
- net Net-(ULED10-Pad4): track 0.00 -> 39.3 mm, vias 0 -> 2
- net Net-(R7-Pad1): track 2.75 -> 41.8 mm
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
Commit message: LED37
Parts:
- K_15: footprint MX_Only:MXOnly-2U-NoLED -> MX_Only:MXOnly-2U-ReversedStabilizers-NoLED
Routing:
- net row0: track 372.3 -> 373.3 mm
- net Net-(ULED13-Pad2): track 70.5 -> 71.3 mm

Commit message: Clean up silkscreen, tracks, and generate gerbers
Parts:
- R1, R6: value 10k -> 10kΩ
- R2, R3: value 5.1k -> 5.1kΩ
- R4, R5: value 22 -> 22Ω
- R7: value 510 ohm -> 510Ω
- SW1: value SW_Push -> RESET
- moved G*** 10.6 mm to (138.5, 93.0)
- moved R1 1.17 mm to (145.4, 49.0), turned to 180 degrees
- moved SW2 0.12 mm to (323.9, 9.60)
- moved K_23 0.08 mm to (153.3, 40.4)
Routing:
- net GND: track 2707.4 -> 2330.0 mm, vias 141 -> 98
- net row1: track 447.3 -> 425.1 mm
- net +5V: track 2370.5 -> 2351.0 mm, vias 91 -> 90
- net Net-(LED52-Pad2): track 55.5 -> 37.6 mm
- net 0col: track 477.8 -> 467.4 mm
- net row2: track 358.4 -> 351.3 mm
- net Net-(ULED12-Pad2): track 49.8 -> 55.8 mm
- net LED: track 223.0 -> 217.6 mm, vias 3 -> 2
- net row8: track 412.4 -> 407.1 mm
- net row4: track 335.2 -> 330.0 mm
- net Net-(LED58-Pad2): track 56.4 -> 51.3 mm
- net Net-(R7-Pad1): track 41.8 -> 36.8 mm
- net Net-(LED23-Pad2): track 73.1 -> 68.7 mm
- net Net-(LED19-Pad2): track 43.5 -> 47.4 mm
- net Net-(LED35-Pad4): track 44.3 -> 41.0 mm
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
Commit message: Fix more traces, regenerate gerbers
Routing:
- net Net-(LED55-Pad4): track 29.2 -> 34.8 mm
- net GND: track 2330.0 -> 2333.1 mm
- net ENC0B: track 279.9 -> 281.2 mm
- net Net-(D_62-Pad2): track 12.0 -> 12.5 mm

Commit message: Add copper fill 0.5
Routing:
- added copper zone on B.Cu, net (none)
- added copper zone on F.Cu, net (none)
Changed lines of the file:
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@@
+    )
+  )
+  (zone (net 0) (net_name "") (layer F.Cu) (hatch edge 0.508)
+    (connect_pads (clearance 0.508))
+    (min_thickness 0.254)
+    (fill yes (arc_segments 32) (thermal_gap 0.508) (thermal_bridge_width 0.508))
+    (polygon
+      (pts
+        (xy -25 -12.75) (xy -24.75 119.25) (xy 355.5 123.5) (xy 355 -12.25)
+      )
+    )
+  )
+  (zone (net 0) (net_name "") (layer B.Cu) (hatch edge 0.508)
+    (connect_pads (clearance 0.508))
+    (min_thickness 0.254)
+    (fill yes (arc_segments 32) (thermal_gap 0.508) (thermal_bridge_width 0.508))
+    (polygon
+      (pts
+        (xy -25 -12.75) (xy -24.75 119.25) (xy 355.5 123.5) (xy 355 -12.25)
+      )
     )
   )
