File: Hardware/Rev 0.5 RGB/trifecta.sch (KiCad schematic (older format))
At the start: 284 parts, among them J1 USB2_C_Receptacle, SW1 SW_Push, SW2 Rotary_Encoder_Switch, SW3 Rotary_Encoder_Switch, SW4 Rotary_Encoder_Switch, U1 ATmega32U4-AU, U2 SRV05-4, Y1 16MHz

Commit message: 08/07
Connections:
- net at ULED5.2 (DOUT): now also ULED6.4 (DIN)
- net at ULED9.4 (DIN): now also ULED8.2 (DOUT)
Changed lines of the file:
@@
-$EndComp
-$Comp
-L power:GND #PWR0157
-U 1 1 5FB8AEBA
-P 25900 5275
-F 0 "#PWR0157" H 25900 5025 50  0001 C CNN
-F 1 "GND" H 25905 5102 50  0000 C CNN
-F 2 "" H 25900 5275 50  0001 C CNN
-F 3 "" H 25900 5275 50  0001 C CNN
-	1    25900 5275
-	1    0    0    -1
 $EndComp
 $Comp
@@
 	25900 6075 25850 6075
 Wire Wire Line
-	25925 5475 25925 5275
-Wire Wire Line
 	25925 5575 25900 5575
 Wire Wire Line
@@
 $EndComp
 Connection ~ 25850 5075
-Connection ~ 25900 5275
 Wire Wire Line
 	25925 2625 25925 2975
@@
 	-1   0    0    -1
 $EndComp
+Wire Wire Line
+	25925 5475 25925 5300
+Wire Wire Line
+	25925 5300 26725 5300
+Wire Wire Line
+	26725 5300 26725 5075
+Wire Wire Line
+	25725 5775 25725 5575
 $EndSCHEMATC

Commit message: LED37
Parts:
- K_15: footprint MX_Only:MXOnly-2U-NoLED -> MX_Only:MXOnly-2U-ReversedStabilizers-NoLED
Changed lines of the file:
@@
 F 0 "K_15" H 18275 8808 60  0000 C CNN
 F 1 "KEYSW" H 18275 8475 60  0001 C CNN
-F 2 "MX_Only:MXOnly-2U-NoLED" H 18275 8575 60  0001 C CNN
+F 2 "MX_Only:MXOnly-2U-ReversedStabilizers-NoLED" H 18275 8575 60  0001 C CNN
 F 3 "" H 18275 8575 60  0000 C CNN
 	1    18275 8575

Commit message: Clean up silkscreen, tracks, and generate gerbers
Parts:
- R1, R6: value 10k -> 10kΩ
- R2, R3: value 5.1k -> 5.1kΩ
- R4, R5: value 22 -> 22Ω
- R7: value 510 ohm -> 510Ω
- SW1: value SW_Push -> RESET
Changed lines of the file:
@@
 EESchema Schematic File Version 4
+LIBS:trifecta-cache
 EELAYER 30 0
 EELAYER END
@@
 P 3350 4100
 F 0 "R5" V 3154 4100 50  0000 C CNN
-F 1 "22" V 3245 4100 50  0000 C CNN
+F 1 "22Ω" V 3245 4100 50  0000 C CNN
 F 2 "Resistor_SMD:R_0805_2012Metric" H 3350 4100 50  0001 C CNN
 F 3 "https://datasheet.lcsc.com/szlcsc/Uniroyal-Elec-0805W8F2202T5E_C17560.pdf" H 3350 4100 50  0001 C CNN
@@
 P 3650 4000
 F 0 "R4" V 3454 4000 50  0000 C CNN
-F 1 "22" V 3545 4000 50  0000 C CNN
+F 1 "22Ω" V 3545 4000 50  0000 C CNN
 F 2 "Resistor_SMD:R_0805_2012Metric" H 3650 4000 50  0001 C CNN
 F 3 "https://datasheet.lcsc.com/szlcsc/Uniroyal-Elec-0805W8F2202T5E_C17560.pdf" H 3650 4000 50  0001 C CNN
@@
 P 4050 2700
 F 0 "R1" H 4109 2746 50  0000 L CNN
-F 1 "10k" H 4109 2655 50  0000 L CNN
+F 1 "10kΩ" H 4109 2655 50  0000 L CNN
 F 2 "Resistor_SMD:R_0805_2012Metric" H 4050 2700 50  0001 C CNN
 F 3 "https://datasheet.lcsc.com/szlcsc/Uniroyal-Elec-0805W8F1002T5E_C17414.pdf" H 4050 2700 50  0001 C CNN
@@
 P 6250 5100
 F 0 "R6" V 6054 5100 50  0000 C CNN
-F 1 "10k" V 6145 5100 50  0000 C CNN
+F 1 "10kΩ" V 6145 5100 50  0000 C CNN
 F 2 "Resistor_SMD:R_0805_2012Metric" H 6250 5100 50  0001 C CNN
 F 3 "https://datasheet.lcsc.com/szlcsc/Uniroyal-Elec-0805W8F1002T5E_C17414.pdf" H 6250 5100 50  0001 C CNN
@@
 P 7750 3250
 F 0 "R2" V 7554 3250 50  0000 C CNN
-F 1 "5.1k" V 7645 3250 50  0000 C CNN
+F 1 "5.1kΩ" V 7645 3250 50  0000 C CNN
 F 2 "Resistor_SMD:R_0805_2012Metric" H 7750 3250 50  0001 C CNN
 F 3 "https://datasheet.lcsc.com/szlcsc/Uniroyal-Elec-0805W8F5101T5E_C27834.pdf" H 7750 3250 50  0001 C CNN
@@
 P 8050 3350
 F 0 "R3" V 7854 3350 50  0000 C CNN
-F 1 "5.1k" V 7945 3350 50  0000 C CNN
+F 1 "5.1kΩ" V 7945 3350 50  0000 C CNN
 F 2 "Resistor_SMD:R_0805_2012Metric" H 8050 3350 50  0001 C CNN
 F 3 "https://datasheet.lcsc.com/szlcsc/Uniroyal-Elec-0805W8F5101T5E_C27834.pdf" H 8050 3350 50  0001 C CNN
@@
 P 3550 3000
 F 0 "SW1" H 3550 3285 50  0000 C CNN
-F 1 "SW_Push" H 3550 3194 50  0000 C CNN
+F 1 "RESET" H 3550 3194 50  0000 C CNN
 F 2 "random-keyboard-parts:SKQG-1155865" H 3550 3200 50  0001 C CNN
 F 3 "~" H 3550 3200 50  0001 C CNN
@@
 P 27675 2625
 F 0 "R7" V 27480 2630 50  0000 C CNN
-F 1 "510 ohm" V 27571 2621 50  0000 C CNN
+F 1 "510Ω" V 27571 2621 50  0000 C CNN
 F 2 "Resistor_SMD:R_0805_2012Metric" H 27675 2625 50  0001 C CNN
 F 3 "https://datasheet.lcsc.com/szlcsc/Uniroyal-Elec-0805W8F5100T5E_C17734.pdf" H 27675 2625 50  0001 C CNN

Commit message: 8/8
Parts:
- added J1: Conn_02x03_Odd_Even, Connector_PinHeader_2.54mm:PinHeader_2x03_P2.54mm_Vertical, symbol conn:Conn_02x03_Odd_Even
Connections:
- net +5V: now also J1.2 (Pin_2)
- net 0col: now also J1.1 (Pin_1)
- net GND: now also J1.6 (Pin_6)
- net col5: now also J1.4 (Pin_4)
- net row3: now also J1.3 (Pin_3)
- new net RESET: J1.5 (Pin_5)
Other:
- moved on the sheet: C1, C11, C13, C16, C9, F1, J1, R1, R2, R3, R4, R5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
