File: Hardware/Rev 0.5 RGB/trifecta.sch (KiCad schematic (older format))
At the start: 285 parts, among them J1 USB2_C_Receptacle, J2 ISP Header, SW1 RESET, SW2 Rotary_Encoder_Switch, SW3 Rotary_Encoder_Switch, SW4 Rotary_Encoder_Switch, U1 ATmega32U4-AU, U2 SRV05-4, Y1 16MHz

Commit message: 8/9
Parts:
- F1: LCSC Part# (none) -> C70068; Mfr (none) -> TECHFUSE; Part# (none) -> nSMD025
- R4, R5: LCSC Part# C17560 -> C17561; Part# 0805W8F2202T5E -> 0805W8F220JT5E
Changed lines of the file:
@@
 F 1 "22Ω" V -355 2825 50  0000 C CNN
 F 2 "Resistor_SMD:R_0805_2012Metric" H -250 2825 50  0001 C CNN
-F 3 "https://datasheet.lcsc.com/szlcsc/Uniroyal-Elec-0805W8F2202T5E_C17560.pdf" H -250 2825 50  0001 C CNN
-F 4 "C17560" V -250 2825 50  0001 C CNN "LCSC Part#"
-F 5 "0805W8F2202T5E" V -250 2825 50  0001 C CNN "Part#"
+F 3 "https://datasheet.lcsc.com/szlcsc/Uniroyal-Elec-0805W8F220JT5E_C17561.pdf" H -250 2825 50  0001 C CNN
+F 4 "C17561" V -250 2825 50  0001 C CNN "LCSC Part#"
+F 5 "0805W8F220JT5E" V -250 2825 50  0001 C CNN "Part#"
 F 6 "Uniroyal Elec" V -250 2825 50  0001 C CNN "Mrf"
 	1    -250 2825
@@
 F 1 "22Ω" V -55 2725 50  0000 C CNN
 F 2 "Resistor_SMD:R_0805_2012Metric" H 50  2725 50  0001 C CNN
-F 3 "https://datasheet.lcsc.com/szlcsc/Uniroyal-Elec-0805W8F2202T5E_C17560.pdf" H 50  2725 50  0001 C CNN
-F 4 "C17560" V 50  2725 50  0001 C CNN "LCSC Part#"
-F 5 "0805W8F2202T5E" V 50  2725 50  0001 C CNN "Part#"
+F 3 "https://datasheet.lcsc.com/szlcsc/Uniroyal-Elec-0805W8F220JT5E_C17561.pdf" H 50  2725 50  0001 C CNN
+F 4 "C17561" V 50  2725 50  0001 C CNN "LCSC Part#"
+F 5 "0805W8F220JT5E" V 50  2725 50  0001 C CNN "Part#"
 F 6 "Uniroyal Elec" V 50  2725 50  0001 C CNN "Mrf"
 	1    50   2725
@@
 F 1 "500mA" V 8536 1075 50  0000 C CNN
 F 2 "Fuse:Fuse_1206_3216Metric" H 8700 875 50  0001 L CNN
-F 3 "~" H 8650 1075 50  0001 C CNN
-F 4 "" V 8650 1075 50  0001 C CNN "LCSC Part#"
-F 5 "" V 8650 1075 50  0001 C CNN "Part#"
-F 6 "" V 8650 1075 50  0001 C CNN "Mfr"
+F 3 "https://datasheet.lcsc.com/szlcsc/TECHFUSE-nSMD025_C70068.pdf" H 8650 1075 50  0001 C CNN
+F 4 "C70068" V 8650 1075 50  0001 C CNN "LCSC Part#"
+F 5 "nSMD025" V 8650 1075 50  0001 C CNN "Part#"
+F 6 "TECHFUSE" V 8650 1075 50  0001 C CNN "Mfr"
 	1    8650 1075
 	0    1    1    0
@@
 Wire Wire Line
 	200  550  200  1725
-Wire Bus Line
-	2500 -225 2500 2250
 Connection ~ 200  1725
 Wire Wire Line
 	200  1725 150  1725
+Wire Bus Line
+	2500 -225 2500 2250
 $EndSCHEMATC
