File: Hardware/Rev 0.5 RGB/trifecta.sch (KiCad schematic (older format))
At the start: 285 parts, among them J1 USB2_C_Receptacle, J2 ISP Header, SW1 RESET, SW2 Rotary_Encoder_Switch, SW3 Rotary_Encoder_Switch, SW4 Rotary_Encoder_Switch, U1 ATmega32U4-AU, U2 SRV05-4, Y1 16MHz

Commit message: 8/8
Connections:
- net RESET: no longer J2.5 (Pin_5)
- net at R1.2, SW1.2, U1.13 (~RESET): now also J2.5 (Pin_5)
Changed lines of the file:
@@
 	450  1325 450  1075
 Wire Wire Line
-	450  1725 150  1725
+	450  1725 200  1725
 Wire Wire Line
 	450  1725 450  1525
@@
 	1    0    0    -1
 $EndComp
-Text GLabel 3075 325  0    50   Input ~ 0
+Text GLabel 1900 175  0    50   Input ~ 0
 RESET
 Wire Wire Line
@@
 Text Label 2625 825  0    50   ~ 0
 MOSI
+Wire Wire Line
+	3075 325  3075 550
+Wire Wire Line
+	3075 550  200  550
+Wire Wire Line
+	200  550  200  1725
 Wire Bus Line
 	2500 -225 2500 2250
+Connection ~ 200  1725
+Wire Wire Line
+	200  1725 150  1725
 $EndSCHEMATC

Commit message: Fix silkscreen + generate gerbers
Parts:
- J2: symbol conn:Conn_02x03_Odd_Even -> trifecta-rescue:Conn_02x03_Odd_Even-conn
Changed lines of the file:
@@
 EESchema Schematic File Version 4
+LIBS:trifecta-cache
 EELAYER 30 0
 EELAYER END
@@
 	25725 5775 25725 5575
 $Comp
-L conn:Conn_02x03_Odd_Even J2
+L trifecta-rescue:Conn_02x03_Odd_Even-conn J2
 U 1 1 5F520C1F
 P 3275 225
@@
 Wire Wire Line
 	200  550  200  1725
-Wire Bus Line
-	2500 -225 2500 2250
 Connection ~ 200  1725
 Wire Wire Line
 	200  1725 150  1725
+Wire Bus Line
+	2500 -225 2500 2250
 $EndSCHEMATC
