File: Hardware/Rev 0.5 RGB Hotswap/trifecta.kicad_pcb (KiCad board)
At the start: 2 copper layers, 361 x 120.8 mm, 280 parts, among them J1 USB2_C_Receptacle, SW1 SW_Push, SW2 Rotary_Encoder_Switch, SW3 Rotary_Encoder_Switch, SW4 Rotary_Encoder_Switch, U1 ATmega32U4-AU, U2 SRV05-4, Y1 16MHz

Commit message: Edit Silkscreens for HS version
TODO: clean up tracks and add silkscreen art
Parts:
- R1, R6: value 10k -> 10kΩ
- R2, R3: value 5.1k -> 5.1kΩ
- R4, R5: value 22 -> 22Ω
- R7: value 510 ohm -> 510Ω
- SW1: value SW_Push -> RESET
- moved R1 1.09 mm to (145.4, 48.9), turned to 180 degrees
Routing:
- net GND: track 2465.6 -> 2406.7 mm, vias 110 -> 103
- net row1: track 446.2 -> 400.5 mm
- net Net-(D_16-Pad2): track 10.1 -> 0.00 mm
- net 0col: track 469.0 -> 463.7 mm
- net row4: track 335.2 -> 330.0 mm
- net row7: track 379.1 -> 377.9 mm
- net +5V: track 2370.3 -> 2371.1 mm, vias 91 -> 90
- net Net-(R1-Pad2): track 38.2 -> 39.0 mm

Commit message: Revert "Edit Silkscreens for HS version"
This reverts commit 5a8b713c0dac6e6c9a90fc558c8fc8e6b1fe5ec3.
Parts:
- R1, R6: value 10kΩ -> 10k
- R2, R3: value 5.1kΩ -> 5.1k
- R4, R5: value 22Ω -> 22
- R7: value 510Ω -> 510 ohm
- SW1: value RESET -> SW_Push
- moved R1 1.09 mm to (144.7, 48.1), turned to 90 degrees
Routing:
- net GND: track 2406.7 -> 2465.6 mm, vias 103 -> 110
- net row1: track 400.5 -> 446.2 mm
- net Net-(D_16-Pad2): track 0.00 -> 10.1 mm
- net 0col: track 463.7 -> 469.0 mm
- net row4: track 330.0 -> 335.2 mm
- net row7: track 377.9 -> 379.1 mm
- net +5V: track 2371.1 -> 2370.3 mm, vias 90 -> 91
- net Net-(R1-Pad2): track 39.0 -> 38.2 mm
