File: Hardware/Rev 0.5 RGB Hotswap/trifecta.kicad_pcb (KiCad board)
At the start: 2 copper layers, 361 x 120.8 mm, 285 parts, among them J1 USB2_C_Receptacle, SW1 SW_Push, SW2 Rotary_Encoder_Switch, SW3 Rotary_Encoder_Switch, SW4 Rotary_Encoder_Switch, U1 ATmega32U4-AU, U2 SRV05-4, Y1 16MHz

Commit message: LED37
Parts:
- removed D_16: D, kbd:D3_SMD_v2
- removed G***: LOGO, graphics:image1
- removed K_14, K_16: KEYSW, MX_Only:MXOnly-1U-NoLED
- removed K_32: KEYSW, MX_Only:MXOnly-1.75U-NoLED
- K_1, K_10, K_11, K_12, K_13, K_18, K_19, K_2, K_20, K_21, K_22, K_23, K_24, K_25, K_26, K_27, K_28, K_29, K_3, K_30, K_31, K_34, K_35, K_36, K_37, K_38, K_39, K_4, K_40, K_41, K_42, K_43, K_44, K_46, K_48, K_49, K_5, K_50, K_51, K_52, K_53, K_54, K_55, K_56, K_57, K_58, K_6, K_60, K_61, K_7, K_70, K_71, K_72, K_8, K_9: footprint MX_Only:MXOnly-1U-NoLED -> MX_Only:MXOnly-1U-Hotswap
- K_15: footprint MX_Only:MXOnly-2U-NoLED -> MX_Only:MXOnly-2U-Hotswap-ReversedStabilizers
- K_17: footprint MX_Only:MXOnly-1.5U-NoLED -> MX_Only:MXOnly-1.5U-Hotswap
- K_33, K_59: footprint MX_Only:MXOnly-1.75U-NoLED -> MX_Only:MXOnly-1.75U-Hotswap
- K_45, K_47, K_66: footprint MX_Only:MXOnly-2.25U-ReversedStabilizers-NoLED -> MX_Only:MXOnly-2.25U-Hotswap-ReversedStabilizers
- K_62, K_63, K_64, K_67, K_68, K_69: footprint MX_Only:MXOnly-1.25U-NoLED -> MX_Only:MXOnly-1.25U-Hotswap
- K_65: footprint MX_Only:MXOnly-2.75U-ReversedStabilizers-NoLED -> MX_Only:MXOnly-2.75U-Hotswap-ReversedStabilizers
Routing:
- net (no net): track 0.00 -> 219.4 mm, vias 0 -> 1
- net col1: track 327.5 -> 218.2 mm, vias 3 -> 8
- net col3: track 231.5 -> 142.8 mm, vias 6 -> 5
- net col2: track 235.5 -> 177.8 mm, vias 2 -> 5
- net GND: track 2707.4 -> 2697.5 mm, vias 141 -> 140
- net Net-(D_33-Pad2): track 17.0 -> 9.08 mm
- net Net-(D_47-Pad2): track 21.2 -> 14.7 mm
- net row3: track 408.9 -> 414.1 mm
- net Net-(D_18-Pad2): track 13.3 -> 8.42 mm
- net col0: track 228.4 -> 232.4 mm, vias 1 -> 6
- net Net-(D_62-Pad2): track 13.2 -> 9.26 mm
- net Net-(D_17-Pad2): track 13.0 -> 9.13 mm
- net Net-(D_4-Pad2): track 11.5 -> 7.70 mm
- net Net-(D_48-Pad2): track 12.9 -> 9.52 mm
- net Net-(D_2-Pad2): track 12.5 -> 9.29 mm
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
Commit message: 8/7 Final
Parts:
- K_31, K_46, K_61: footprint MX_Only:MXOnly-1U-Hotswap -> MX_Only:MXOnly-1U-NoLED
Routing:
- net GND: track 2697.5 -> 2465.6 mm, vias 140 -> 110
- net (no net): track 219.4 -> 0.00 mm, vias 1 -> 0
- net col3: track 142.8 -> 246.1 mm, vias 5 -> 13
- net col1: track 218.2 -> 319.7 mm, vias 8 -> 13
- net col2: track 177.8 -> 239.4 mm, vias 5 -> 11
- net row6: track 354.4 -> 333.7 mm
- net col4: track 256.4 -> 236.3 mm, vias 2 -> 11
- net Net-(D_15-Pad2): track 31.0 -> 16.2 mm
- net row0: track 372.3 -> 386.8 mm
- net row8: track 412.4 -> 402.9 mm
- net 0col: track 477.8 -> 469.0 mm, vias 1 -> 7
- net Net-(D_66-Pad2): track 22.1 -> 13.8 mm
- net Net-(D_45-Pad2): track 21.2 -> 13.9 mm
- net Net-(D_65-Pad2): track 21.8 -> 14.7 mm
- net Net-(D_26-Pad2): track 13.3 -> 7.05 mm
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
Commit message: Clean up silkscreens, regenerate gerbers
Parts:
- R1, R6: value 10k -> 10kΩ
- R2, R3: value 5.1k -> 5.1kΩ
- R4, R5: value 22 -> 22Ω
- R7: value 510 ohm -> 510Ω
- SW1: value SW_Push -> RESET
- moved R1 1.17 mm to (145.4, 49.0), turned to 180 degrees
- moved SW2 0.26 mm to (324.0, 9.50)
Routing:
- net GND: track 2465.6 -> 2406.7 mm, vias 110 -> 103
- net row1: track 446.2 -> 400.5 mm
- net Net-(D_16-Pad2): track 10.1 -> 0.00 mm
- net 0col: track 469.0 -> 463.7 mm
- net row4: track 335.2 -> 330.0 mm
- net row7: track 379.1 -> 377.9 mm
- net Net-(R1-Pad2): track 38.2 -> 39.0 mm
- net +5V: track 2370.3 -> 2371.1 mm, vias 91 -> 90
