File: Hardware/Rev 0.5 RGB Hotswap/trifecta.sch (KiCad schematic (older format))
At the start: 280 parts, among them J1 USB2_C_Receptacle, SW1 RESET, SW2 Rotary_Encoder_Switch, SW3 Rotary_Encoder_Switch, SW4 Rotary_Encoder_Switch, U1 ATmega32U4-AU, U2 SRV05-4, Y1 16MHz

Commit message: Revert "Edit Silkscreens for HS version"
This reverts commit 5a8b713c0dac6e6c9a90fc558c8fc8e6b1fe5ec3.
Parts:
- R1, R6: value 10kΩ -> 10k
- R2, R3: value 5.1kΩ -> 5.1k
- R4, R5: value 22Ω -> 22
- R7: value 510Ω -> 510 ohm
- SW1: value RESET -> SW_Push
Changed lines of the file:
@@
 EESchema Schematic File Version 4
-LIBS:trifecta-cache
 EELAYER 30 0
 EELAYER END
@@
 P 3350 4100
 F 0 "R5" V 3154 4100 50  0000 C CNN
-F 1 "22Ω" V 3245 4100 50  0000 C CNN
+F 1 "22" V 3245 4100 50  0000 C CNN
 F 2 "Resistor_SMD:R_0805_2012Metric" H 3350 4100 50  0001 C CNN
 F 3 "https://datasheet.lcsc.com/szlcsc/Uniroyal-Elec-0805W8F2202T5E_C17560.pdf" H 3350 4100 50  0001 C CNN
@@
 P 3650 4000
 F 0 "R4" V 3454 4000 50  0000 C CNN
-F 1 "22Ω" V 3545 4000 50  0000 C CNN
+F 1 "22" V 3545 4000 50  0000 C CNN
 F 2 "Resistor_SMD:R_0805_2012Metric" H 3650 4000 50  0001 C CNN
 F 3 "https://datasheet.lcsc.com/szlcsc/Uniroyal-Elec-0805W8F2202T5E_C17560.pdf" H 3650 4000 50  0001 C CNN
@@
 P 4050 2700
 F 0 "R1" H 4109 2746 50  0000 L CNN
-F 1 "10kΩ" H 4109 2655 50  0000 L CNN
+F 1 "10k" H 4109 2655 50  0000 L CNN
 F 2 "Resistor_SMD:R_0805_2012Metric" H 4050 2700 50  0001 C CNN
 F 3 "https://datasheet.lcsc.com/szlcsc/Uniroyal-Elec-0805W8F1002T5E_C17414.pdf" H 4050 2700 50  0001 C CNN
@@
 P 6250 5100
 F 0 "R6" V 6054 5100 50  0000 C CNN
-F 1 "10kΩ" V 6145 5100 50  0000 C CNN
+F 1 "10k" V 6145 5100 50  0000 C CNN
 F 2 "Resistor_SMD:R_0805_2012Metric" H 6250 5100 50  0001 C CNN
 F 3 "https://datasheet.lcsc.com/szlcsc/Uniroyal-Elec-0805W8F1002T5E_C17414.pdf" H 6250 5100 50  0001 C CNN
@@
 P 7750 3250
 F 0 "R2" V 7554 3250 50  0000 C CNN
-F 1 "5.1kΩ" V 7645 3250 50  0000 C CNN
+F 1 "5.1k" V 7645 3250 50  0000 C CNN
 F 2 "Resistor_SMD:R_0805_2012Metric" H 7750 3250 50  0001 C CNN
 F 3 "https://datasheet.lcsc.com/szlcsc/Uniroyal-Elec-0805W8F5101T5E_C27834.pdf" H 7750 3250 50  0001 C CNN
@@
 P 8050 3350
 F 0 "R3" V 7854 3350 50  0000 C CNN
-F 1 "5.1kΩ" V 7945 3350 50  0000 C CNN
+F 1 "5.1k" V 7945 3350 50  0000 C CNN
 F 2 "Resistor_SMD:R_0805_2012Metric" H 8050 3350 50  0001 C CNN
 F 3 "https://datasheet.lcsc.com/szlcsc/Uniroyal-Elec-0805W8F5101T5E_C27834.pdf" H 8050 3350 50  0001 C CNN
@@
 P 3550 3000
 F 0 "SW1" H 3550 3285 50  0000 C CNN
-F 1 "RESET" H 3550 3194 50  0000 C CNN
+F 1 "SW_Push" H 3550 3194 50  0000 C CNN
 F 2 "random-keyboard-parts:SKQG-1155865" H 3550 3200 50  0001 C CNN
 F 3 "~" H 3550 3200 50  0001 C CNN
@@
 P 27675 2625
 F 0 "R7" V 27480 2630 50  0000 C CNN
-F 1 "510Ω" V 27571 2621 50  0000 C CNN
+F 1 "510 ohm" V 27571 2621 50  0000 C CNN
 F 2 "Resistor_SMD:R_0805_2012Metric" H 27675 2625 50  0001 C CNN
 F 3 "https://datasheet.lcsc.com/szlcsc/Uniroyal-Elec-0805W8F5100T5E_C17734.pdf" H 27675 2625 50  0001 C CNN
