File: Hardware/Rev 0.5 RGB Hotswap/trifecta.sch (KiCad schematic (older format))
At the start: 284 parts, among them J1 USB2_C_Receptacle, SW1 SW_Push, SW2 Rotary_Encoder_Switch, SW3 Rotary_Encoder_Switch, SW4 Rotary_Encoder_Switch, U1 ATmega32U4-AU, U2 SRV05-4, Y1 16MHz

Commit message: LED37
Parts:
- removed D_16: D, kbd:D3_SMD_v2, symbol trifecta-rescue:D_Small-Device-unnamed-rescue
- removed K_14, K_16: KEYSW, MX_Only:MXOnly-1U-NoLED, symbol MX_Alps_Hybrid:MX-NoLED
- removed K_32: KEYSW, MX_Only:MXOnly-1.75U-NoLED, symbol MX_Alps_Hybrid:MX-NoLED
- K_1, K_10, K_11, K_12, K_13, K_18, K_19, K_2, K_20, K_21, K_22, K_23, K_24, K_25, K_26, K_27, K_28, K_29, K_3, K_30, K_31, K_34, K_35, K_36, K_37, K_38, K_39, K_4, K_40, K_41, K_42, K_43, K_44, K_46, K_48, K_49, K_5, K_50, K_51, K_52, K_53, K_54, K_55, K_56, K_57, K_58, K_6, K_60, K_61, K_7, K_70, K_71, K_72, K_8, K_9: footprint MX_Only:MXOnly-1U-NoLED -> MX_Only:MXOnly-1U-Hotswap
- K_15: footprint MX_Only:MXOnly-2U-NoLED -> MX_Only:MXOnly-2U-Hotswap-ReversedStabilizers
- K_17: footprint MX_Only:MXOnly-1.5U-NoLED -> MX_Only:MXOnly-1.5U-Hotswap
- K_33, K_59: footprint MX_Only:MXOnly-1.75U-NoLED -> MX_Only:MXOnly-1.75U-Hotswap
- K_45, K_47, K_66: footprint MX_Only:MXOnly-2.25U-ReversedStabilizers-NoLED -> MX_Only:MXOnly-2.25U-Hotswap-ReversedStabilizers
- K_62, K_63, K_64, K_67, K_68, K_69: footprint MX_Only:MXOnly-1.25U-NoLED -> MX_Only:MXOnly-1.25U-Hotswap
- K_65: footprint MX_Only:MXOnly-2.75U-ReversedStabilizers-NoLED -> MX_Only:MXOnly-2.75U-Hotswap-ReversedStabilizers

Commit message: 8/7 Final
Parts:
- K_31, K_46, K_61: footprint MX_Only:MXOnly-1U-Hotswap -> MX_Only:MXOnly-1U-NoLED
Changed lines of the file:
@@
 F 0 "K_31" H 19275 9808 60  0000 C CNN
 F 1 "KEYSW" H 19275 9475 60  0001 C CNN
-F 2 "MX_Only:MXOnly-1U-Hotswap" H 19275 9575 60  0001 C CNN
+F 2 "MX_Only:MXOnly-1U-NoLED" H 19275 9575 60  0001 C CNN
 F 3 "" H 19275 9575 60  0000 C CNN
 	1    19275 9575
@@
 F 0 "K_46" H 19275 10808 60  0000 C CNN
 F 1 "KEYSW" H 19275 10475 60  0001 C CNN
-F 2 "MX_Only:MXOnly-1U-Hotswap" H 19275 10575 60  0001 C CNN
+F 2 "MX_Only:MXOnly-1U-NoLED" H 19275 10575 60  0001 C CNN
 F 3 "" H 19275 10575 60  0000 C CNN
 	1    19275 10575
@@
 F 0 "K_61" H 19275 11808 60  0000 C CNN
 F 1 "KEYSW" H 19275 11475 60  0001 C CNN
-F 2 "MX_Only:MXOnly-1U-Hotswap" H 19275 11575 60  0001 C CNN
+F 2 "MX_Only:MXOnly-1U-NoLED" H 19275 11575 60  0001 C CNN
 F 3 "" H 19275 11575 60  0000 C CNN
 	1    19275 11575

Commit message: Clean up silkscreens, regenerate gerbers
Parts:
- R1, R6: value 10k -> 10kΩ
- R2, R3: value 5.1k -> 5.1kΩ
- R4, R5: value 22 -> 22Ω
- R7: value 510 ohm -> 510Ω
- SW1: value SW_Push -> RESET
Changed lines of the file:
@@
 EESchema Schematic File Version 4
+LIBS:trifecta-cache
 EELAYER 30 0
 EELAYER END
@@
 P 3350 4100
 F 0 "R5" V 3154 4100 50  0000 C CNN
-F 1 "22" V 3245 4100 50  0000 C CNN
+F 1 "22Ω" V 3245 4100 50  0000 C CNN
 F 2 "Resistor_SMD:R_0805_2012Metric" H 3350 4100 50  0001 C CNN
 F 3 "https://datasheet.lcsc.com/szlcsc/Uniroyal-Elec-0805W8F2202T5E_C17560.pdf" H 3350 4100 50  0001 C CNN
@@
 P 3650 4000
 F 0 "R4" V 3454 4000 50  0000 C CNN
-F 1 "22" V 3545 4000 50  0000 C CNN
+F 1 "22Ω" V 3545 4000 50  0000 C CNN
 F 2 "Resistor_SMD:R_0805_2012Metric" H 3650 4000 50  0001 C CNN
 F 3 "https://datasheet.lcsc.com/szlcsc/Uniroyal-Elec-0805W8F2202T5E_C17560.pdf" H 3650 4000 50  0001 C CNN
@@
 P 4050 2700
 F 0 "R1" H 4109 2746 50  0000 L CNN
-F 1 "10k" H 4109 2655 50  0000 L CNN
+F 1 "10kΩ" H 4109 2655 50  0000 L CNN
 F 2 "Resistor_SMD:R_0805_2012Metric" H 4050 2700 50  0001 C CNN
 F 3 "https://datasheet.lcsc.com/szlcsc/Uniroyal-Elec-0805W8F1002T5E_C17414.pdf" H 4050 2700 50  0001 C CNN
@@
 P 6250 5100
 F 0 "R6" V 6054 5100 50  0000 C CNN
-F 1 "10k" V 6145 5100 50  0000 C CNN
+F 1 "10kΩ" V 6145 5100 50  0000 C CNN
 F 2 "Resistor_SMD:R_0805_2012Metric" H 6250 5100 50  0001 C CNN
 F 3 "https://datasheet.lcsc.com/szlcsc/Uniroyal-Elec-0805W8F1002T5E_C17414.pdf" H 6250 5100 50  0001 C CNN
@@
 P 7750 3250
 F 0 "R2" V 7554 3250 50  0000 C CNN
-F 1 "5.1k" V 7645 3250 50  0000 C CNN
+F 1 "5.1kΩ" V 7645 3250 50  0000 C CNN
 F 2 "Resistor_SMD:R_0805_2012Metric" H 7750 3250 50  0001 C CNN
 F 3 "https://datasheet.lcsc.com/szlcsc/Uniroyal-Elec-0805W8F5101T5E_C27834.pdf" H 7750 3250 50  0001 C CNN
@@
 P 8050 3350
 F 0 "R3" V 7854 3350 50  0000 C CNN
-F 1 "5.1k" V 7945 3350 50  0000 C CNN
+F 1 "5.1kΩ" V 7945 3350 50  0000 C CNN
 F 2 "Resistor_SMD:R_0805_2012Metric" H 8050 3350 50  0001 C CNN
 F 3 "https://datasheet.lcsc.com/szlcsc/Uniroyal-Elec-0805W8F5101T5E_C27834.pdf" H 8050 3350 50  0001 C CNN
@@
 P 3550 3000
 F 0 "SW1" H 3550 3285 50  0000 C CNN
-F 1 "SW_Push" H 3550 3194 50  0000 C CNN
+F 1 "RESET" H 3550 3194 50  0000 C CNN
 F 2 "random-keyboard-parts:SKQG-1155865" H 3550 3200 50  0001 C CNN
 F 3 "~" H 3550 3200 50  0001 C CNN
@@
 P 27675 2625
 F 0 "R7" V 27480 2630 50  0000 C CNN
-F 1 "510 ohm" V 27571 2621 50  0000 C CNN
+F 1 "510Ω" V 27571 2621 50  0000 C CNN
 F 2 "Resistor_SMD:R_0805_2012Metric" H 27675 2625 50  0001 C CNN
 F 3 "https://datasheet.lcsc.com/szlcsc/Uniroyal-Elec-0805W8F5100T5E_C17734.pdf" H 27675 2625 50  0001 C CNN

Commit message: 8/8
Parts:
- added J2: ISP Header, Connector_PinHeader_2.54mm:PinHeader_2x03_P2.54mm_Vertical, symbol conn:Conn_02x03_Odd_Even
Connections:
- net +5V: now also J2.2 (Pin_2)
- net 0col: now also J2.1 (Pin_1)
- net GND: now also J2.6 (Pin_6)
- net col5: now also J2.4 (Pin_4)
- net row3: now also J2.3 (Pin_3)
- net at R1.2, SW1.2, U1.13 (~RESET): now also J2.5 (Pin_5)
Other:
- moved on the sheet: F1, J1, R2, R3

Commit message: 8/10
Parts:
- F1: LCSC Part# (none) -> C70068; Mfr (none) -> TECHFUSE; Part# (none) -> nSMD025
- R4, R5: LCSC Part# C17560 -> C17561; Part# 0805W8F2202T5E -> 0805W8F220JT5E
Changed lines of the file:
@@
 F 1 "22Ω" V 3245 4100 50  0000 C CNN
 F 2 "Resistor_SMD:R_0805_2012Metric" H 3350 4100 50  0001 C CNN
-F 3 "https://datasheet.lcsc.com/szlcsc/Uniroyal-Elec-0805W8F2202T5E_C17560.pdf" H 3350 4100 50  0001 C CNN
-F 4 "C17560" V 3350 4100 50  0001 C CNN "LCSC Part#"
-F 5 "0805W8F2202T5E" V 3350 4100 50  0001 C CNN "Part#"
+F 3 "https://datasheet.lcsc.com/szlcsc/Uniroyal-Elec-0805W8F220JT5E_C17561.pdf" H 3350 4100 50  0001 C CNN
+F 4 "C17561" V 3350 4100 50  0001 C CNN "LCSC Part#"
+F 5 "0805W8F220JT5E" V 3350 4100 50  0001 C CNN "Part#"
 F 6 "Uniroyal Elec" V 3350 4100 50  0001 C CNN "Mrf"
 	1    3350 4100
@@
 F 1 "22Ω" V 3545 4000 50  0000 C CNN
 F 2 "Resistor_SMD:R_0805_2012Metric" H 3650 4000 50  0001 C CNN
-F 3 "https://datasheet.lcsc.com/szlcsc/Uniroyal-Elec-0805W8F2202T5E_C17560.pdf" H 3650 4000 50  0001 C CNN
-F 4 "C17560" V 3650 4000 50  0001 C CNN "LCSC Part#"
-F 5 "0805W8F2202T5E" V 3650 4000 50  0001 C CNN "Part#"
+F 3 "https://datasheet.lcsc.com/szlcsc/Uniroyal-Elec-0805W8F220JT5E_C17561.pdf" H 3650 4000 50  0001 C CNN
+F 4 "C17561" V 3650 4000 50  0001 C CNN "LCSC Part#"
+F 5 "0805W8F220JT5E" V 3650 4000 50  0001 C CNN "Part#"
 F 6 "Uniroyal Elec" V 3650 4000 50  0001 C CNN "Mrf"
 	1    3650 4000
@@
 F 1 "500mA" V -864 7675 50  0000 C CNN
 F 2 "Fuse:Fuse_1206_3216Metric" H -700 7475 50  0001 L CNN
-F 3 "~" H -750 7675 50  0001 C CNN
-F 4 "" V -750 7675 50  0001 C CNN "LCSC Part#"
-F 5 "" V -750 7675 50  0001 C CNN "Part#"
-F 6 "" V -750 7675 50  0001 C CNN "Mfr"
+F 3 "https://datasheet.lcsc.com/szlcsc/TECHFUSE-nSMD025_C70068.pdf" H -750 7675 50  0001 C CNN
+F 4 "C70068" V -750 7675 50  0001 C CNN "LCSC Part#"
+F 5 "nSMD025" V -750 7675 50  0001 C CNN "Part#"
+F 6 "TECHFUSE" V -750 7675 50  0001 C CNN "Mfr"
 	1    -750 7675
 	0    1    1    0
@@
 Wire Wire Line
 	6100 3300 6800 3300
-Wire Bus Line
-	6000 1225 6000 3525
 Text Label 5725 3100 0    50   ~ 0
 SCK
@@
 Text Label 6125 3300 0    50   ~ 0
 MISO
+Wire Bus Line
+	6000 1225 6000 3525
 $EndSCHEMATC
