File: Hardware/Rev0.5rgb/trifecta.kicad_pcb (KiCad board)
At the start: 2 copper layers, 361 x 128 mm, 286 parts, among them J1 USB2_C_Receptacle, J2 ISP Header, SW1 RESET, SW2 Rotary_Encoder_Switch, SW3 Rotary_Encoder_Switch, SW4 Rotary_Encoder_Switch, U1 ATmega32U4-AU, U2 SRV05-4, Y1 16MHz

Commit message: 8/21-4
Other:
- rule pad_to_mask_clearance: 0 -> 0.01

Commit message: 9/6
Parts:
- moved C44 13.7 mm to (271.7, 61.2)
- moved D_29 13.7 mm to (292.4, 36.9)
- moved SW3 13.7 mm to (341.2, 37.8)
- moved K_29 13.7 mm to (284.1, 34.0)
- moved K_30 13.7 mm to (307.9, 34.0)
- moved C1 13.7 mm to (148.3, 50.4)
- moved C28 13.7 mm to (264.9, 42.1)
- moved C58 13.7 mm to (265.1, 80.2)
- moved C77 13.7 mm to (151.3, 115.5)
- moved D_24 13.7 mm to (193.5, 44.7)
- moved D_55 13.7 mm to (214.2, 80.1)
- moved D_56 13.7 mm to (232.9, 76.5)
- moved D_68 13.7 mm to (261.4, 95.2)
- moved K_56 13.7 mm to (224.1, 74.4)
- moved K_58 13.7 mm to (265.0, 72.1)
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