File: Hardware/Rev0.6rgb/trifecta.kicad_pcb (KiCad board)
At the start: 2 copper layers, 361 x 128 mm, 285 parts, among them J1 USB2_C_Receptacle, J2 ISP Header, SW1 RESET, SW2 Rotary_Encoder_Switch, SW3 Rotary_Encoder_Switch, SW4 Rotary_Encoder_Switch, U1 ATmega32U4-AU, U2 SRV05-4, Y1 16MHz

Commit message: 10/16
Parts:
- added K_52: KEYSW, MX_Only:MXOnly-1U-NoLED, F.Cu at (131.7, 85.5)
- K_30: footprint MX_Only:MXOnly-1.5U-NoLED -> MX_Only:MXOnly-1U-NoLED
- ULED1: footprint LED_kicad_footprints-master:Underglow YS-SK6812MINI-E -> LED_SMD:LED_SK6812MINI_PLCC4_3.5x3.5mm_P1.75mm
- moved ULED1 2.85 mm to (352.3, 9.16)
- moved D_2 2.73 mm to (51.8, 17.7)
- moved C2 2.66 mm to (43.9, 23.0)
- moved LED2 2.59 mm to (43.9, 20.4)
- moved D_3 1.94 mm to (70.8, 17.8), turned to 90 degrees
- moved LED3 1.21 mm to (62.5, 18.2), turned to 0 degrees
- moved C4 0.60 mm to (81.3, 24.6), turned to 348 degrees
- moved LED4 0.47 mm to (81.9, 22.1), turned to 168 degrees
Routing:
- net col1: track 214.5 -> 258.5 mm
- net (no net): track 115.5 -> 78.4 mm
- net Net-(LED2-Pad4): track 45.6 -> 26.0 mm
- net +5V: track 2386.9 -> 2393.8 mm
- net GND: track 2455.0 -> 2450.4 mm
- net col0: track 229.3 -> 225.5 mm
- net row1: track 423.1 -> 419.3 mm
- net Net-(D_2-Pad2): track 12.5 -> 9.36 mm
- net Net-(LED18-Pad4): track 36.7 -> 39.3 mm
- net row0: track 373.3 -> 371.2 mm
- net Net-(LED19-Pad2): track 47.4 -> 48.5 mm
- net Net-(ULED1-Pad2): track 77.5 -> 78.4 mm
- net Net-(R7-Pad1): track 36.8 -> 37.6 mm

Commit message: 10/16-2
Parts:
- moved C18 3.41 mm to (49.3, 42.0)
- moved LED17 3.40 mm to (25.4, 39.4)
- moved LED18 3.32 mm to (49.2, 39.4)
- moved D_17 2.98 mm to (33.3, 37.5)
- moved D_18 2.82 mm to (57.0, 36.9)
- moved LED33 1.20 mm to (23.7, 58.5)
- moved LED34 1.13 mm to (49.9, 58.5)
- moved C34 1.12 mm to (49.9, 61.1)
- moved D_34 0.87 mm to (57.9, 56.9)
Routing:
- net col0: track 225.5 -> 232.1 mm
- net +5V: track 2393.8 -> 2399.5 mm
- net col1: track 258.5 -> 263.6 mm
- net Net-(D_18-Pad2): track 13.3 -> 8.41 mm
- net Net-(LED17-Pad4): track 32.9 -> 37.7 mm
- net Net-(LED18-Pad4): track 39.3 -> 34.9 mm
- net Net-(LED34-Pad2): track 39.9 -> 43.0 mm
- net row3: track 456.6 -> 453.5 mm
- net row2: track 351.3 -> 348.8 mm
- net Net-(D_33-Pad2): track 17.0 -> 15.2 mm
- net GND: track 2450.4 -> 2448.9 mm
- net Net-(LED1-Pad4): track 37.1 -> 38.6 mm
- net Net-(D_17-Pad2): track 12.7 -> 11.3 mm
- net Net-(LED18-Pad2): track 38.1 -> 39.5 mm
- net Net-(LED33-Pad4): track 34.1 -> 35.3 mm
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
Commit message: 10/16-3
Parts:
- removed G***: LOGO, graphics:image1
- ULED10, ULED11, ULED12, ULED13, ULED14, ULED2, ULED3, ULED4, ULED5, ULED6, ULED7, ULED8, ULED9: footprint LED_kicad_footprints-master:Underglow YS-SK6812MINI-E -> LED_SMD:LED_SK6812MINI_PLCC4_3.5x3.5mm_P1.75mm
- moved C30 3.52 mm to (304.6, 42.1)
- moved LED30 3.29 mm to (304.6, 39.6)
- moved C12 3.07 mm to (248.4, 20.8)
- moved ULED13 2.98 mm to (268.2, 3.38)
- moved ULED7 2.96 mm to (7.38, 10.6)
- moved LED12 2.91 mm to (248.4, 18.3)
- moved D_13 2.84 mm to (275.2, 18.8)
- moved LED65 2.79 mm to (115.0, 107.1), turned to 348 degrees
- moved D_12 2.75 mm to (256.3, 17.2)
- moved LED64 2.73 mm to (77.5, 99.0), turned to 348 degrees
- moved LED13 2.66 mm to (267.1, 20.4)
- moved LED15 2.61 mm to (295.7, 20.4)
- moved C15 2.60 mm to (295.7, 22.9)
- moved LED52 2.47 mm to (130.5, 90.9), turned to 168 degrees
- moved ULED14 2.43 mm to (323.2, 27.7)
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Routing:
- net +5V: track 2399.5 -> 2477.9 mm, vias 92 -> 96
- net Net-(LED22-Pad2): track 38.1 -> 0.00 mm, vias 2 -> 0
- net Net-(LED52-Pad2): track 37.6 -> 0.00 mm, vias 2 -> 0
- net row0: track 371.2 -> 399.1 mm, vias 5 -> 7
- net Net-(LED12-Pad4): track 27.9 -> 0.00 mm, vias 2 -> 0
- net Net-(D_18-Pad2): track 8.41 -> 10.5 mm
- net row3: track 453.5 -> 455.4 mm
- net Net-(ULED6-Pad2): track 135.1 -> 136.6 mm
- net Net-(ULED8-Pad2): track 38.1 -> 39.6 mm
- net Net-(ULED7-Pad2): track 55.8 -> 56.6 mm
