File: Hardware/Rev0.6rgb/trifecta.kicad_pcb (KiCad board)
At the start: 2 copper layers, 361 x 128 mm, 285 parts, among them J1 USB2_C_Receptacle, J2 ISP Header, SW1 RESET, SW2 Rotary_Encoder_Switch, SW3 Rotary_Encoder_Switch, SW4 Rotary_Encoder_Switch, U1 ATmega32U4-AU, U2 SRV05-4, Y1 16MHz

Commit message: Trifecta Board
Parts:
- moved D_27 4.06 mm to (251.2, 35.3)
- moved D_28 3.74 mm to (269.9, 36.4)
- moved C67 3.25 mm to (224.9, 101.6), turned to 12 degrees
- moved LED28 3.22 mm to (261.7, 39.4)
- moved C28 3.20 mm to (261.7, 42.0)
- moved C66 3.17 mm to (192.0, 108.5), turned to 12 degrees
- moved LED66 3.15 mm to (191.5, 106.1), turned to 192 degrees
- moved LED67 3.14 mm to (224.3, 99.1), turned to 192 degrees
- moved LED29 3.10 mm to (280.8, 39.5)
- moved ULED6 3.04 mm to (59.3, 87.8)
- moved LED27 3.01 mm to (243.1, 38.4)
- moved ULED2 2.94 mm to (346.4, 77.5)
- moved ULED4 2.94 mm to (237.4, 86.8)
- moved ULED11 2.68 mm to (190.5, 9.14)
- moved D_67 2.58 mm to (231.7, 96.1), turned to 102 degrees
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Routing:
- net row3: track 455.4 -> 583.2 mm
- net (no net): track 78.4 -> 0.00 mm
- net col1: track 263.6 -> 333.9 mm, vias 3 -> 4
- net row8: track 407.1 -> 366.8 mm
- net Net-(LED22-Pad2): track 0.00 -> 39.0 mm, vias 0 -> 2
- net Net-(LED52-Pad2): track 0.00 -> 35.6 mm, vias 0 -> 2
- net GND: track 2449.4 -> 2479.2 mm, vias 107 -> 108
- net Net-(LED12-Pad4): track 0.00 -> 29.7 mm
- net row0: track 399.1 -> 373.6 mm, vias 7 -> 5
- net +5V: track 2477.9 -> 2452.9 mm, vias 96 -> 92
- net Net-(LED35-Pad4): track 41.0 -> 29.5 mm
- net row4: track 330.0 -> 340.2 mm
- net col3: track 230.7 -> 239.4 mm
- net Net-(D_66-Pad2): track 22.1 -> 14.2 mm
- net Net-(LED54-Pad2): track 32.6 -> 25.5 mm
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- removed copper zone on B.Cu, net (none)
- removed copper zone on F.Cu, net (none)
- removed copper zone on F.Cu, net GND

Commit message: Trifecta Keyboard
Routing:
- added copper zone on B.Cu, net (none)
- added copper zone on F.Cu, net (none)
- added copper zone on F.Cu, net GND
Changed lines of the file:
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@@
+    )
+  )
+  (zone (net 73) (net_name GND) (layer F.Cu) (hatch edge 0.508)
+    (connect_pads (clearance 0.508))
+    (min_thickness 0.254)
+    (fill yes (arc_segments 32) (thermal_gap 0.508) (thermal_bridge_width 0.508))
+    (polygon
+      (pts
+        (xy 371.53088 133.0452) (xy 151.21382 133.0452) (xy -3.53822 118.11508) (xy -3.53822 -14.33322) (xy 371.53088 -14.33322)
+      )
+    )
+  )
+  (zone (net 0) (net_name "") (layer F.Cu) (hatch edge 0.508)
+    (connect_pads (clearance 0.508))
+    (min_thickness 0.254)
+    (fill yes (arc_segments 32) (thermal_gap 0.508) (thermal_bridge_width 0.508))
+    (polygon
+      (pts
+        (xy 371.04828 132.96392) (xy 147.4343 132.96392) (xy -3.06578 119.37492) (xy -3.06578 -11.87704) (xy -3.60172 -14.43482)
+        (xy 371.04828 -16.256)
+      )
+    )
+  )
+  (zone (net 73) (net_name GND) (layer B.Cu) (hatch edge 0.508)
+    (connect_pads (clearance 0.508))
+    (min_thickness 0.254)
+    (fill yes (arc_segments 32) (thermal_gap 0.508) (thermal_bridge_width 0.508))
+    (polygon
+      (pts
+        (xy 370.9543 -16.15694) (xy 370.9543 132.03428) (xy 160.97504 133.51002) (xy -3.73126 119.23268) (xy -3.73126 -14.42466)
+        (xy -3.7338 -17.12722)
+      )
+    )
+  )
+  (zone (net 0) (net_name "") (layer B.Cu) (hatch edge 0.508)
+    (connect_pads (clearance 0.508))
+    (min_thickness 0.254)
+    (fill yes (arc_segments 32) (thermal_gap 0.508) (thermal_bridge_width 0.508))
+    (polygon
+      (pts
+        (xy 371.46738 -16.76146) (xy 371.17274 132.1181) (xy 158.1912 132.70992) (xy -3.38328 118.78056) (xy -3.07848 -15.21714)
+        (xy -3.24104 -18.16862)
+      )
     )
   )
