File: Hardware/Rev0.6rgb/trifecta.sch (KiCad schematic (older format))
At the start: 285 parts, among them J1 USB2_C_Receptacle, J2 ISP Header, SW1 RESET, SW2 Rotary_Encoder_Switch, SW3 Rotary_Encoder_Switch, SW4 Rotary_Encoder_Switch, U1 ATmega32U4-AU, U2 SRV05-4, Y1 16MHz

Commit message: 10/16-3
Parts:
- ULED1, ULED10, ULED11, ULED12, ULED13, ULED14, ULED2, ULED3, ULED4, ULED5, ULED6, ULED7, ULED8, ULED9: footprint LED_kicad_footprints-master:Underglow YS-SK6812MINI-E -> LED_SMD:LED_SK6812MINI_PLCC4_3.5x3.5mm_P1.75mm
Changed lines of the file:
@@
 F 0 "ULED13" H 25325 3252 50  0000 C CNN
 F 1 "YS-SK6812MINI-E" H 25325 3343 50  0000 C CNN
-F 2 "LED_kicad_footprints-master:Underglow YS-SK6812MINI-E" H 25325 3175 50  0001 C CNN
+F 2 "LED_SMD:LED_SK6812MINI_PLCC4_3.5x3.5mm_P1.75mm" H 25325 3175 50  0001 C CNN
 F 3 "http://www.world-semi.com/uploads/soft/150522/1-150522091P5.pdf" H 25325 3425 50  0001 C CNN
 	1    25325 3475
@@
 F 0 "ULED12" H 25325 3752 50  0000 C CNN
 F 1 "YS-SK6812MINI-E" H 25325 3843 50  0000 C CNN
-F 2 "LED_kicad_footprints-master:Underglow YS-SK6812MINI-E" H 25325 3675 50  0001 C CNN
+F 2 "LED_SMD:LED_SK6812MINI_PLCC4_3.5x3.5mm_P1.75mm" H 25325 3675 50  0001 C CNN
 F 3 "http://www.world-semi.com/uploads/soft/150522/1-150522091P5.pdf" H 25325 3925 50  0001 C CNN
 	1    25325 3975
@@
 F 0 "ULED11" H 25325 4252 50  0000 C CNN
 F 1 "YS-SK6812MINI-E" H 25325 4343 50  0000 C CNN
-F 2 "LED_kicad_footprints-master:Underglow YS-SK6812MINI-E" H 25325 4175 50  0001 C CNN
+F 2 "LED_SMD:LED_SK6812MINI_PLCC4_3.5x3.5mm_P1.75mm" H 25325 4175 50  0001 C CNN
 F 3 "http://www.world-semi.com/uploads/soft/150522/1-150522091P5.pdf" H 25325 4425 50  0001 C CNN
 	1    25325 4475
@@
 F 0 "ULED10" H 25325 4752 50  0000 C CNN
 F 1 "YS-SK6812MINI-E" H 25325 4843 50  0000 C CNN
-F 2 "LED_kicad_footprints-master:Underglow YS-SK6812MINI-E" H 25325 4675 50  0001 C CNN
+F 2 "LED_SMD:LED_SK6812MINI_PLCC4_3.5x3.5mm_P1.75mm" H 25325 4675 50  0001 C CNN
 F 3 "http://www.world-semi.com/uploads/soft/150522/1-150522091P5.pdf" H 25325 4925 50  0001 C CNN
 	1    25325 4975
@@
 F 0 "ULED1" H 26325 2852 50  0000 C CNN
 F 1 "YS-SK6812MINI-E" H 26325 2943 50  0000 C CNN
-F 2 "LED_kicad_footprints-master:Underglow YS-SK6812MINI-E" H 26325 2775 50  0001 C CNN
+F 2 "LED_SMD:LED_SK6812MINI_PLCC4_3.5x3.5mm_P1.75mm" H 26325 2775 50  0001 C CNN
 F 3 "http://www.world-semi.com/uploads/soft/150522/1-150522091P5.pdf" H 26325 3025 50  0001 C CNN
 	1    26325 3075
@@
 F 0 "ULED2" H 26325 3352 50  0000 C CNN
 F 1 "YS-SK6812MINI-E" H 26325 3443 50  0000 C CNN
-F 2 "LED_kicad_footprints-master:Underglow YS-SK6812MINI-E" H 26325 3275 50  0001 C CNN
+F 2 "LED_SMD:LED_SK6812MINI_PLCC4_3.5x3.5mm_P1.75mm" H 26325 3275 50  0001 C CNN
 F 3 "http://www.world-semi.com/uploads/soft/150522/1-150522091P5.pdf" H 26325 3525 50  0001 C CNN
 	1    26325 3575
@@
 F 0 "ULED3" H 26325 3852 50  0000 C CNN
 F 1 "YS-SK6812MINI-E" H 26325 3943 50  0000 C CNN
-F 2 "LED_kicad_footprints-master:Underglow YS-SK6812MINI-E" H 26325 3775 50  0001 C CNN
+F 2 "LED_SMD:LED_SK6812MINI_PLCC4_3.5x3.5mm_P1.75mm" H 26325 3775 50  0001 C CNN
 F 3 "http://www.world-semi.com/uploads/soft/150522/1-150522091P5.pdf" H 26325 4025 50  0001 C CNN
 	1    26325 4075
@@
 F 0 "ULED4" H 26325 4352 50  0000 C CNN
 F 1 "YS-SK6812MINI-E" H 26325 4443 50  0000 C CNN
-F 2 "LED_kicad_footprints-master:Underglow YS-SK6812MINI-E" H 26325 4275 50  0001 C CNN
+F 2 "LED_SMD:LED_SK6812MINI_PLCC4_3.5x3.5mm_P1.75mm" H 26325 4275 50  0001 C CNN
 F 3 "http://www.world-semi.com/uploads/soft/150522/1-150522091P5.pdf" H 26325 4525 50  0001 C CNN
 	1    26325 4575
@@
 F 0 "ULED5" H 26325 4852 50  0000 C CNN
 F 1 "YS-SK6812MINI-E" H 26325 4943 50  0000 C CNN
-F 2 "LED_kicad_footprints-master:Underglow YS-SK6812MINI-E" H 26325 4775 50  0001 C CNN
+F 2 "LED_SMD:LED_SK6812MINI_PLCC4_3.5x3.5mm_P1.75mm" H 26325 4775 50  0001 C CNN
 F 3 "http://www.world-semi.com/uploads/soft/150522/1-150522091P5.pdf" H 26325 5025 50  0001 C CNN
 	1    26325 5075
@@
 F 0 "ULED9" H 25325 5252 50  0000 C CNN
 F 1 "YS-SK6812MINI-E" H 25325 5343 50  0000 C CNN
-F 2 "LED_kicad_footprints-master:Underglow YS-SK6812MINI-E" H 25325 5175 50  0001 C CNN
+F 2 "LED_SMD:LED_SK6812MINI_PLCC4_3.5x3.5mm_P1.75mm" H 25325 5175 50  0001 C CNN
 F 3 "http://www.world-semi.com/uploads/soft/150522/1-150522091P5.pdf" H 25325 5425 50  0001 C CNN
 	1    25325 5475
@@
 F 0 "ULED8" H 25325 5752 50  0000 C CNN
 F 1 "YS-SK6812MINI-E" H 25325 5843 50  0000 C CNN
-F 2 "LED_kicad_footprints-master:Underglow YS-SK6812MINI-E" H 25325 5675 50  0001 C CNN
+F 2 "LED_SMD:LED_SK6812MINI_PLCC4_3.5x3.5mm_P1.75mm" H 25325 5675 50  0001 C CNN
 F 3 "http://www.world-semi.com/uploads/soft/150522/1-150522091P5.pdf" H 25325 5925 50  0001 C CNN
 	1    25325 5975
@@
 F 0 "ULED6" H 26325 5352 50  0000 C CNN
 F 1 "YS-SK6812MINI-E" H 26325 5443 50  0000 C CNN
-F 2 "LED_kicad_footprints-master:Underglow YS-SK6812MINI-E" H 26325 5275 50  0001 C CNN
+F 2 "LED_SMD:LED_SK6812MINI_PLCC4_3.5x3.5mm_P1.75mm" H 26325 5275 50  0001 C CNN
 F 3 "http://www.world-semi.com/uploads/soft/150522/1-150522091P5.pdf" H 26325 5525 50  0001 C CNN
 	1    26325 5575
@@
 F 0 "ULED7" H 26325 5852 50  0000 C CNN
 F 1 "YS-SK6812MINI-E" H 26325 5943 50  0000 C CNN
-F 2 "LED_kicad_footprints-master:Underglow YS-SK6812MINI-E" H 26325 5775 50  0001 C CNN
+F 2 "LED_SMD:LED_SK6812MINI_PLCC4_3.5x3.5mm_P1.75mm" H 26325 5775 50  0001 C CNN
 F 3 "http://www.world-semi.com/uploads/soft/150522/1-150522091P5.pdf" H 26325 6025 50  0001 C CNN
 	1    26325 6075
@@
 F 0 "ULED14" H 25325 2752 50  0000 C CNN
 F 1 "YS-SK6812MINI-E" H 25325 2843 50  0000 C CNN
-F 2 "LED_kicad_footprints-master:Underglow YS-SK6812MINI-E" H 25325 2675 50  0001 C CNN
+F 2 "LED_SMD:LED_SK6812MINI_PLCC4_3.5x3.5mm_P1.75mm" H 25325 2675 50  0001 C CNN
 F 3 "http://www.world-semi.com/uploads/soft/150522/1-150522091P5.pdf" H 25325 2925 50  0001 C CNN
 	1    25325 2975
@@
 Wire Wire Line
 	200  1725 150  1725
-Wire Bus Line
-	2500 -225 2500 2250
 $Comp
 L trifecta-rescue:WS2812B-Worldsemi-unnamed-rescue LED15
@@
 Text Notes 9975 3050 0    50   ~ 0
 79
+Wire Bus Line
+	2500 -225 2500 2250
 $EndSCHEMATC
